Commit message: fix something

File: src/robots/cyberdog_description/urdf/cyberdog_description.urdf (robot description, URDF)
Before this commit: robot cyberdog_description, 19 links, 18 joints
Links:
- link trunk: mass 7.18 -> 7.18+1.6

Commit message: fix cyberdog model

File: src/robots/cyberdog_description/urdf/cyberdog_description.urdf (robot description, URDF)
Before this commit: robot cyberdog_description, 19 links, 18 joints
Links:
- added link FL_thigh_shoulder
- added link FR_thigh_shoulder
- added link RL_thigh_shoulder
- added link RR_thigh_shoulder
- link FL_calf: geometry collision mesh filename=package://cyberdog_description/meshes/calf.STL; visual mesh filename=package://cyberdog_description/meshes/calf.STL scale=1 1 1
- link FL_foot: geometry collision sphere radius=0.025; visual sphere radius=0.025
- link FL_hip: geometry collision mesh filename=package://cyberdog_description/meshes/hip.STL; visual mesh filename=package://cyberdog_description/meshes/hip.STL scale=1 1 1
- link FL_thigh: geometry collision mesh filename=package://cyberdog_description/meshes/thigh.STL; visual mesh filename=package://cyberdog_description/meshes/thigh.STL scale=1 1 1
- link FR_calf: geometry collision mesh filename=package://cyberdog_description/meshes/calf.STL; visual mesh filename=package://cyberdog_description/meshes/calf.STL scale=1 1 1
- link FR_foot: geometry collision sphere radius=0.025; visual sphere radius=0.025
- link FR_hip: geometry collision mesh filename=package://cyberdog_description/meshes/hip_mirror.STL; visual mesh filename=package://cyberdog_description/meshes/hip_mirror.STL scale=1 1 1
- link FR_thigh: geometry collision mesh filename=package://cyberdog_description/meshes/thigh.STL; visual mesh filename=package://cyberdog_description/meshes/thigh.STL scale=1 1 1
- link RL_calf: geometry collision mesh filename=package://cyberdog_description/meshes/calf.STL; visual mesh filename=package://cyberdog_description/meshes/calf.STL scale=1 1 1
- link RL_foot: geometry collision sphere radius=0.025; visual sphere radius=0.025
- link RL_hip: geometry collision mesh filename=package://cyberdog_description/meshes/hip.STL; visual mesh filename=package://cyberdog_description/meshes/hip.STL scale=1 1 1
- link RL_thigh: geometry collision mesh filename=package://cyberdog_description/meshes/thigh.STL; visual mesh filename=package://cyberdog_description/meshes/thigh.STL scale=1 1 1
- link RR_calf: geometry collision mesh filename=package://cyberdog_description/meshes/calf.STL; visual mesh filename=package://cyberdog_description/meshes/calf.STL scale=1 1 1
- link RR_foot: geometry collision sphere radius=0.025; visual sphere radius=0.025
- link RR_hip: geometry collision mesh filename=package://cyberdog_description/meshes/hip_mirror.STL; visual mesh filename=package://cyberdog_description/meshes/hip_mirror.STL scale=1 1 1
- link RR_thigh: geometry collision mesh filename=package://cyberdog_description/meshes/thigh.STL; visual mesh filename=package://cyberdog_description/meshes/thigh.STL scale=1 1 1
- link imu_link: mass None -> 0.001; geometry visual box size=0.001 0.001 0.001
- link trunk: mass 7.18+1.6 -> 8.78; geometry collision mesh filename=package://cyberdog_description/meshes/trunk.STL; visual mesh filename=package://cyberdog_description/meshes/trunk.STL scale=1 1 1
Joints:
- added joint FL_hip_fixed: type fixed, parent FL_hip, child FL_thigh_shoulder, origin xyz=0 0.10 0 rpy=0 0 0
- added joint FR_hip_fixed: type fixed, parent FR_hip, child FR_thigh_shoulder, origin xyz=0 -0.10 0 rpy=0 0 0
- added joint RL_hip_fixed: type fixed, parent RL_hip, child RL_thigh_shoulder, origin xyz=0 0.10 0 rpy=0 0 0
- added joint RR_hip_fixed: type fixed, parent RR_hip, child RR_thigh_shoulder, origin xyz=0 -0.10 0 rpy=0 0 0
- joint FL_calf_joint: limit lower=-2.478 upper=-0.506 effort=240 velocity=12 -> lower=-2.478 upper=-0.506 effort=24 velocity=12
- joint FL_hip_joint: limit lower=-0.75 upper=0.75 effort=170 velocity=12 -> lower=-0.75 upper=0.75 effort=17 velocity=12
- joint FL_thigh_joint: limit lower=-1.257 upper=4.363 effort=240 velocity=12 -> lower=-1.257 upper=4.363 effort=24 velocity=12
- joint FR_calf_joint: limit lower=-2.478 upper=-0.506 effort=240 velocity=12 -> lower=-2.478 upper=-0.506 effort=24 velocity=12
- joint FR_hip_joint: limit lower=-0.75 upper=0.75 effort=170 velocity=12 -> lower=-0.75 upper=0.75 effort=17 velocity=12
- joint FR_thigh_joint: limit lower=-1.257 upper=4.363 effort=240 velocity=12 -> lower=-1.257 upper=4.363 effort=24 velocity=12
- joint RL_calf_joint: limit lower=-2.478 upper=-0.506 effort=240 velocity=12 -> lower=-2.478 upper=-0.506 effort=24 velocity=12
- joint RL_hip_joint: limit lower=-0.75 upper=0.75 effort=170 velocity=12 -> lower=-0.75 upper=0.75 effort=17 velocity=12
- joint RL_thigh_joint: limit lower=-2.01 upper=3.49 effort=240 velocity=12 -> lower=-2.01 upper=3.49 effort=24 velocity=12
- joint RR_calf_joint: limit lower=-2.478 upper=-0.506 effort=240 velocity=12 -> lower=-2.478 upper=-0.506 effort=24 velocity=12
- joint RR_hip_joint: limit lower=-0.75 upper=0.75 effort=170 velocity=12 -> lower=-0.75 upper=0.75 effort=17 velocity=12
- joint RR_thigh_joint: limit lower=-2.01 upper=3.49 effort=240 velocity=12 -> lower=-2.01 upper=3.49 effort=24 velocity=12

Commit message: add new cyberdog model

File: src/robots/cyberdog_description/urdf/cyberdog_description.urdf (robot description, URDF)
Before this commit: robot cyberdog_description, 23 links, 22 joints
Links:
- added link FL_calf_rotor, mass 0.076506382
- added link FL_hip_rotor, mass 0.076506382
- added link FL_thigh_rotor, mass 0.076506382
- added link FR_calf_rotor, mass 0.076506382
- added link FR_hip_rotor, mass 0.076506382
- added link FR_thigh_rotor, mass 0.076506382
- added link RL_calf_rotor, mass 0.076506382
- added link RL_hip_rotor, mass 0.076506382
- added link RL_thigh_rotor, mass 0.076506382
- added link RR_calf_rotor, mass 0.076506382
- added link RR_hip_rotor, mass 0.076506382
- added link RR_thigh_rotor, mass 0.076506382
- link FL_calf: mass 0.114 -> 0.1135916; geometry collision box size=0.016 0.016 0.209; collision sphere radius=0.016
- link FL_foot: mass 0.026 -> None; geometry collision sphere radius=0.018; visual sphere radius=0.018
- link FL_hip: mass 0.509 -> 0.537806728; geometry collision cylinder length=0.052 radius=0.047; visual cylinder length=0.052 radius=0.047
- link FL_thigh: mass 0.664 -> 0.950266218; geometry collision box size=0.2 0.035 0.05; visual box size=0.2 0.035 0.05
- link FL_thigh_shoulder: geometry collision cylinder length=0.052 radius=0.047; visual cylinder length=0.052 radius=0.047
- link FR_calf: mass 0.114 -> 0.1135916; geometry collision box size=0.016 0.016 0.209; collision sphere radius=0.016
- link FR_foot: mass 0.026 -> None; geometry collision sphere radius=0.018; visual sphere radius=0.018
- link FR_hip: mass 0.509 -> 0.537806728; geometry collision cylinder length=0.052 radius=0.047; visual cylinder length=0.052 radius=0.047
- link FR_thigh: mass 0.664 -> 0.950266218; geometry collision box size=0.2 0.035 0.05; visual box size=0.2 0.035 0.05
- link FR_thigh_shoulder: geometry collision cylinder length=0.052 radius=0.047; visual cylinder length=0.052 radius=0.047
- link RL_calf: mass 0.114 -> 0.1135916; geometry collision box size=0.016 0.016 0.209; collision sphere radius=0.016
- link RL_foot: mass 0.026 -> None; geometry collision sphere radius=0.018; visual sphere radius=0.018
- link RL_hip: mass 0.509 -> 0.537806728; geometry collision cylinder length=0.052 radius=0.047; visual cylinder length=0.052 radius=0.047
- link RL_thigh: mass 0.664 -> 0.950266218; geometry collision box size=0.2 0.035 0.05; visual box size=0.2 0.035 0.05
- link RL_thigh_shoulder: geometry collision cylinder length=0.052 radius=0.047; visual cylinder length=0.052 radius=0.047
- link RR_calf: mass 0.114 -> 0.1135916; geometry collision box size=0.016 0.016 0.209; collision sphere radius=0.016
- link RR_foot: mass 0.026 -> None; geometry collision sphere radius=0.018; visual sphere radius=0.018
- link RR_hip: mass 0.509 -> 0.537806728; geometry collision cylinder length=0.052 radius=0.047; visual cylinder length=0.052 radius=0.047
- link RR_thigh: mass 0.664 -> 0.950266218; geometry collision box size=0.2 0.035 0.05; visual box size=0.2 0.035 0.05
- link RR_thigh_shoulder: geometry collision cylinder length=0.052 radius=0.047; visual cylinder length=0.052 radius=0.047
- link imu_link: mass 0.001 -> None; geometry 
- link trunk: mass 8.78 -> 6.248410872; geometry collision box size=0.36 0.23 0.15; visual box size=0.36 0.23 0.15
Joints:
- added joint FL_calf_rotor_fix: type fixed, parent FL_thigh, child FL_calf_rotor, origin xyz=0 -0.0426259 0 rpy=0 0 0
- added joint FL_hip_rotor_fix: type fixed, parent FL_hip, child FL_hip_rotor, origin xyz=-0.0832504 0 0 rpy=0 0 0
- added joint FL_thigh_rotor_fix: type fixed, parent FL_thigh, child FL_thigh_rotor, origin xyz=0 -0.107226 0 rpy=0 0 0
- added joint FR_calf_rotor_fix: type fixed, parent FR_thigh, child FR_calf_rotor, origin xyz=0 0.0426259 0 rpy=0 0 0
- added joint FR_hip_rotor_fix: type fixed, parent FR_hip, child FR_hip_rotor, origin xyz=-0.0832504 0 0 rpy=0 0 0
- added joint FR_thigh_rotor_fix: type fixed, parent FR_thigh, child FR_thigh_rotor, origin xyz=0 0.107226 0 rpy=0 0 0
- added joint RL_calf_rotor_fix: type fixed, parent RL_thigh, child RL_calf_rotor, origin xyz=0 -0.0426259 0 rpy=0 0 0
- added joint RL_hip_rotor_fix: type fixed, parent RL_hip, child RL_hip_rotor, origin xyz=0.0832504 0 0 rpy=0 0 0
- added joint RL_thigh_rotor_fix: type fixed, parent RL_thigh, child RL_thigh_rotor, origin xyz=0 -0.107226 0 rpy=0 0 0
- added joint RR_calf_rotor_fix: type fixed, parent RR_thigh, child RR_calf_rotor, origin xyz=0 0.0426259 0 rpy=0 0 0
- added joint RR_hip_rotor_fix: type fixed, parent RR_hip, child RR_hip_rotor, origin xyz=0.0832504 0 0 rpy=0 0 0
- added joint RR_thigh_rotor_fix: type fixed, parent RR_thigh, child RR_thigh_rotor, origin xyz=0 0.107226 0 rpy=0 0 0
- joint FL_calf_joint: limit lower=-2.478 upper=-0.506 effort=24 velocity=12 -> lower=-2.49582083035 upper=-0.717155789644 effort=24 velocity=31
- joint FL_foot_fixed: origin xyz=0 0 -0.217 rpy=0 0 0 -> xyz=0 0 -0.19999999999999998 rpy=0 0 0
- joint FL_hip_fixed: origin xyz=0 0.10 0 rpy=0 0 0 -> xyz=0 0.053076000000000005 0 rpy=0 0 0
- joint FL_hip_joint: limit lower=-0.75 upper=0.75 effort=17 velocity=12 -> lower=-0.76096355387 upper=0.76096355387 effort=24 velocity=31; origin xyz=0.23536 0.05 0 rpy=0 0 0 -> xyz=0.23035 0.05 0 rpy=0 0 0
- joint FL_thigh_joint: limit lower=-1.257 upper=4.363 effort=24 velocity=12 -> lower=-1.88495559215 upper=3.76991118431 effort=24 velocity=31; origin xyz=0 0.10715 0 rpy=0 0 0 -> xyz=0 0.105076 0 rpy=0 0 0
- joint FR_calf_joint: limit lower=-2.478 upper=-0.506 effort=24 velocity=12 -> lower=-2.49582083035 upper=-0.717155789644 effort=24 velocity=31
- joint FR_foot_fixed: origin xyz=0 0 -0.217 rpy=0 0 0 -> xyz=0 0 -0.19999999999999998 rpy=0 0 0
- joint FR_hip_fixed: origin xyz=0 -0.10 0 rpy=0 0 0 -> xyz=0 -0.053076000000000005 0 rpy=0 0 0
- joint FR_hip_joint: limit lower=-0.75 upper=0.75 effort=17 velocity=12 -> lower=-0.76096355387 upper=0.76096355387 effort=24 velocity=31; origin xyz=0.23536 -0.05 0 rpy=0 0 0 -> xyz=0.23035 -0.05 0 rpy=0 0 0
- joint FR_thigh_joint: limit lower=-1.257 upper=4.363 effort=24 velocity=12 -> lower=-1.88495559215 upper=3.76991118431 effort=24 velocity=31; origin xyz=0 -0.10715 0 rpy=0 0 0 -> xyz=0 -0.105076 0 rpy=0 0 0
- joint RL_calf_joint: limit lower=-2.478 upper=-0.506 effort=24 velocity=12 -> lower=-2.49582083035 upper=-0.717155789644 effort=24 velocity=31
- joint RL_foot_fixed: origin xyz=0 0 -0.217 rpy=0 0 0 -> xyz=0 0 -0.19999999999999998 rpy=0 0 0
- joint RL_hip_fixed: origin xyz=0 0.10 0 rpy=0 0 0 -> xyz=0 0.053076000000000005 0 rpy=0 0 0
- joint RL_hip_joint: limit lower=-0.75 upper=0.75 effort=17 velocity=12 -> lower=-0.76096355387 upper=0.76096355387 effort=24 velocity=31; origin xyz=-0.23536 0.05 0 rpy=0 0 0 -> xyz=-0.23035 0.05 0 rpy=0 0 0
- joint RL_thigh_joint: limit lower=-2.01 upper=3.49 effort=24 velocity=12 -> lower=-1.88495559215 upper=3.76991118431 effort=24 velocity=31; origin xyz=0 0.10715 0 rpy=0 0 0 -> xyz=0 0.105076 0 rpy=0 0 0
- joint RR_calf_joint: limit lower=-2.478 upper=-0.506 effort=24 velocity=12 -> lower=-2.49582083035 upper=-0.717155789644 effort=24 velocity=31
- joint RR_foot_fixed: origin xyz=0 0 -0.217 rpy=0 0 0 -> xyz=0 0 -0.19999999999999998 rpy=0 0 0
- joint RR_hip_fixed: origin xyz=0 -0.10 0 rpy=0 0 0 -> xyz=0 -0.053076000000000005 0 rpy=0 0 0
- joint RR_hip_joint: limit lower=-0.75 upper=0.75 effort=17 velocity=12 -> lower=-0.76096355387 upper=0.76096355387 effort=24 velocity=31; origin xyz=-0.23536 -0.05 0 rpy=0 0 0 -> xyz=-0.23035 -0.05 0 rpy=0 0 0
- joint RR_thigh_joint: limit lower=-2.01 upper=3.49 effort=24 velocity=12 -> lower=-1.88495559215 upper=3.76991118431 effort=24 velocity=31; origin xyz=0 -0.10715 0 rpy=0 0 0 -> xyz=0 -0.105076 0 rpy=0 0 0
