Commit message: fix cyberdog model

File: src/robots/cyberdog1_description/urdf/cyberdog_description.urdf (robot description, URDF)
Before this commit: robot cyberdog_description, 35 links, 34 joints
Links:
- link imu_link: mass None -> 0.001; geometry visual box size=0.001 0.001 0.001

File: src/robots/cyberdog1_description/xacro/gazebo.xacro (robot description, xacro)
@@ -9,5 +9,5 @@
     </gazebo>
     <!-- Show the trajectory of trunk center. -->
-    <gazebo>
+    <!-- <gazebo>
         <plugin name="3dplot" filename="libLinkPlot3DPlugin.so">
             <frequency>10</frequency>
@@ -18,5 +18,5 @@
             </plot>
         </plugin>
-    </gazebo>
+    </gazebo> -->
     <!-- Show the trajectory of foot. You can add another trajectory about another foot. -->
     <!-- <gazebo>

File: src/robots/cyberdog1_description/xacro/leg.xacro (robot description, xacro)
@@ -61,5 +61,5 @@
             </inertial>
         </link>
-        <joint name="${name}_hip_rotor_fix" type="fixed">
+        <joint name="${name}_hip_rotor_fix" type="fixed" dont_collapse="true">
             <origin rpy="0 0 0" xyz="${-abad_rotor_offset*front_hind} 0 0" />
             <parent link="${name}_hip" />
@@ -146,5 +146,5 @@
             </inertial>
         </link>
-        <joint name="${name}_thigh_rotor_fix" type="fixed">
+        <joint name="${name}_thigh_rotor_fix" type="fixed" dont_collapse="true">
             <origin rpy="0 0 0" xyz="0 ${hip_rotor_offset*mirror} 0" />
             <parent link="${name}_thigh" />
@@ -159,5 +159,5 @@
             </inertial>
         </link>
-        <joint name="${name}_calf_rotor_fix" type="fixed">
+        <joint name="${name}_calf_rotor_fix" type="fixed" dont_collapse="true">
             <origin rpy="0 0 0" xyz="0 ${knee_rotor_offset*mirror} 0" />
             <parent link="${name}_thigh" />

File: src/robots/cyberdog1_description/xacro/robot.xacro (robot description, xacro)
@@ -78,5 +78,5 @@
     </joint>
     <link name="imu_link">
-        <!-- <inertial>
+        <inertial>
             <mass value="0.001" />
             <origin rpy="0 0 0" xyz="0 0 0" />
@@ -88,6 +88,7 @@
                 <box size="0.001 0.001 0.001" />
             </geometry>
+            <material name="red"/>
         </visual>
-        <collision>
+        <!-- <collision>
             <origin rpy="0 0 0" xyz="0 0 0" />
             <geometry>
