Commit message: fix: add gazebo config to b2w urdf

File: src/robots/b2w_description/urdf/b2w_description.urdf (robot description, URDF)
Before this commit: robot b2w_description, 26 links, 25 joints
Links:
- removed link base_link
- added link base; visual box size=0.001 0.001 0.001
- added link trunk, mass 35.606; collision box size=0.5 0.28 0.15; visual mesh filename=package://b2w_description/meshes/base_link.dae
Joints:
- added joint floating_base: type fixed, parent base, child trunk, origin xyz=0 0 0 rpy=0 0 0
- joint FL_hip_joint: parent base_link -> trunk
- joint FR_hip_joint: parent base_link -> trunk
- joint RL_hip_joint: parent base_link -> trunk
- joint RR_hip_joint: parent base_link -> trunk
- joint f_oc_link: parent base_link -> trunk
- joint joint_f_dc: parent base_link -> trunk
- joint joint_head: parent base_link -> trunk
- joint joint_imu: parent base_link -> trunk
- joint joint_lidar: parent base_link -> trunk
- joint joint_logo: parent base_link -> trunk
- joint joint_r_dc: parent base_link -> trunk
- joint joint_r_oc: parent base_link -> trunk
- joint joint_tail: parent base_link -> trunk
