Commit message: l4w4

File: src/robots/l4w4_description/urdf/l4w4.urdf (robot description, URDF)
Before this commit: robot l4w4, 17 links, 16 joints
Links:
- added link base; visual box size=0.001 0.001 0.001
- added link imu_link, mass 0
- link FL_calf: geometry collision box size=0.06 0.03 0.1; visual mesh filename=package://l4w4_description/meshes/shank_R.STL scale=1 -1 1
- link FL_foot: geometry collision cylinder length=0.038 radius=0.105; visual mesh filename=package://l4w4_description/meshes/wheel_R.STL scale=1 -1 1
- link FL_hip: geometry collision cylinder length=0 radius=0; visual mesh filename=package://l4w4_description/meshes/shoulder_R.STL scale=1 -1 1
- link FL_thigh: geometry collision box size=0.122 0.044 0.32; visual mesh filename=package://l4w4_description/meshes/thigh_R.STL scale=1 -1 1
- link FR_calf: geometry collision box size=0.06 0.03 0.1; visual mesh filename=package://l4w4_description/meshes/shank_R.STL scale=1 1 1
- link FR_foot: geometry collision cylinder length=0.038 radius=0.105; visual mesh filename=package://l4w4_description/meshes/wheel_R.STL scale=1 1 1
- link FR_hip: geometry collision cylinder length=0 radius=0; visual mesh filename=package://l4w4_description/meshes/shoulder_R.STL
- link FR_thigh: geometry collision box size=0.122 0.044 0.32; visual mesh filename=package://l4w4_description/meshes/thigh_R.STL scale=1 1 1
- link RL_calf: geometry collision box size=0.06 0.03 0.1; visual mesh filename=package://l4w4_description/meshes/shank_R.STL scale=1 -1 1
- link RL_foot: geometry collision cylinder length=0.038 radius=0.105; visual mesh filename=package://l4w4_description/meshes/wheel_R.STL scale=1 -1 1
- link RL_hip: geometry collision cylinder length=0 radius=0; visual mesh filename=package://l4w4_description/meshes/shoulder_R.STL scale=-1 -1 1
- link RL_thigh: geometry collision box size=0.122 0.044 0.32; visual mesh filename=package://l4w4_description/meshes/thigh_R.STL scale=1 -1 1
- link RR_calf: geometry collision box size=0.06 0.03 0.1; visual mesh filename=package://l4w4_description/meshes/shank_R.STL scale=1 1 1
- link RR_foot: geometry collision cylinder length=0.038 radius=0.105; visual mesh filename=package://l4w4_description/meshes/wheel_R.STL scale=1 1 1
- link RR_hip: geometry collision cylinder length=0 radius=0; visual mesh filename=package://l4w4_description/meshes/shoulder_R.STL scale=-1 1 1
- link RR_thigh: geometry collision box size=0.122 0.044 0.32; visual mesh filename=package://l4w4_description/meshes/thigh_R.STL scale=1 1 1
- link trunk: geometry collision box size=0.688 0.18 0.18; visual mesh filename=package://l4w4_description/meshes/trunk.STL
Joints:
- added joint floating_base: type fixed, parent base, child trunk, origin xyz=0 0 0 rpy=0 0 0
- added joint imu_joint: type fixed, parent trunk, child imu_link, origin xyz=0 0 0 rpy=0 0 0
- joint FL_hip_joint: limit lower=-0.785 upper=0.785 effort=130 velocity=11.5 -> lower=-0.5236 upper=0.5236 effort=110 velocity=11.5
- joint FL_thigh_joint: limit lower=-1.4 upper=3.14 effort=135 velocity=12.56 -> lower=-1.4 upper=3.14 effort=110 velocity=12.56
- joint FR_hip_joint: limit lower=-0.785 upper=0.785 effort=130 velocity=11.5 -> lower=-0.5236 upper=0.5236 effort=110 velocity=11.5
- joint FR_thigh_joint: limit lower=-1.4 upper=3.14 effort=135 velocity=12.56 -> lower=-1.4 upper=3.14 effort=110 velocity=12.56
- joint RL_hip_joint: limit lower=-0.785 upper=0.785 effort=130 velocity=11.5 -> lower=-0.5236 upper=0.5236 effort=110 velocity=11.5
- joint RL_thigh_joint: limit lower=-1.4 upper=3.14 effort=135 velocity=12.56 -> lower=-1.4 upper=3.14 effort=110 velocity=12.56
- joint RR_hip_joint: limit lower=-0.785 upper=0.785 effort=130 velocity=11.5 -> lower=-0.5236 upper=0.5236 effort=110 velocity=11.5
- joint RR_thigh_joint: limit lower=-1.4 upper=3.14 effort=135 velocity=12.56 -> lower=-1.4 upper=3.14 effort=110 velocity=12.56

Commit message: fix bugs

File: src/robots/l4w4_description/urdf/l4w4.urdf (robot description, URDF)
Before this commit: robot l4w4, 19 links, 18 joints
Links:
- link FL_foot: mass 1.939 -> 2.6; geometry collision cylinder length=0.040 radius=0.105; visual mesh filename=package://l4w4_description/meshes/wheel_R.STL scale=1 -1 1
- link FR_foot: mass 1.939 -> 2.6; geometry collision cylinder length=0.040 radius=0.105; visual mesh filename=package://l4w4_description/meshes/wheel_R.STL scale=1 1 1
- link RL_foot: mass 1.939 -> 2.6; geometry collision cylinder length=0.040 radius=0.105; visual mesh filename=package://l4w4_description/meshes/wheel_R.STL scale=1 -1 1
- link RR_foot: mass 1.939 -> 2.6; geometry collision cylinder length=0.040 radius=0.105; visual mesh filename=package://l4w4_description/meshes/wheel_R.STL scale=1 1 1
Joints:
- joint RR_foot_joint: limit lower=-1000000 upper=1000000 effort=32 velocity=12.56 -> lower=-1000000 upper=1000000 effort=32 velocity=12.0
