Commit message: fix: update g1_description

File: src/robots/g1_description/urdf/g1_12dof.urdf (robot description, URDF)
Before this commit: robot g1_23dof_rev_1_0, 32 links, 31 joints
Joints:
- joint left_elbow_joint: type revolute -> fixed
- joint left_shoulder_pitch_joint: type revolute -> fixed
- joint left_shoulder_roll_joint: type revolute -> fixed
- joint left_shoulder_yaw_joint: type revolute -> fixed
- joint left_wrist_roll_joint: type revolute -> fixed
- joint right_elbow_joint: type revolute -> fixed
- joint right_shoulder_pitch_joint: type revolute -> fixed
- joint right_shoulder_roll_joint: type revolute -> fixed
- joint right_shoulder_yaw_joint: type revolute -> fixed
- joint right_wrist_roll_joint: type revolute -> fixed
- joint waist_yaw_joint: type revolute -> fixed

File: src/robots/g1_description/urdf/g1_23dof_rev_1_0.urdf (robot description, URDF)
Before this commit: robot g1_23dof_rev_1_0, 32 links, 31 joints
Links:
- removed link base
- link head_link: geometry collision mesh filename=meshes/head_link.STL; visual mesh filename=meshes/head_link.STL
- link left_ankle_pitch_link: geometry collision mesh filename=meshes/left_ankle_pitch_link.STL; visual mesh filename=meshes/left_ankle_pitch_link.STL
- link left_ankle_roll_link: geometry collision sphere radius=0.005; collision sphere radius=0.005
- link left_elbow_link: geometry collision mesh filename=meshes/left_elbow_link.STL; visual mesh filename=meshes/left_elbow_link.STL
- link left_hip_pitch_link: geometry collision mesh filename=meshes/left_hip_pitch_link.STL; visual mesh filename=meshes/left_hip_pitch_link.STL
- link left_hip_roll_link: geometry collision mesh filename=meshes/left_hip_roll_link.STL; visual mesh filename=meshes/left_hip_roll_link.STL
- link left_hip_yaw_link: geometry collision mesh filename=meshes/left_hip_yaw_link.STL; visual mesh filename=meshes/left_hip_yaw_link.STL
- link left_knee_link: geometry collision mesh filename=meshes/left_knee_link.STL; visual mesh filename=meshes/left_knee_link.STL
- link left_shoulder_pitch_link: geometry collision cylinder length=0.05 radius=0.03; visual mesh filename=meshes/left_shoulder_pitch_link.STL
- link left_shoulder_roll_link: geometry collision cylinder length=0.03 radius=0.03; visual mesh filename=meshes/left_shoulder_roll_link.STL
- link left_shoulder_yaw_link: geometry collision mesh filename=meshes/left_shoulder_yaw_link.STL; visual mesh filename=meshes/left_shoulder_yaw_link.STL
- link left_wrist_roll_rubber_hand: geometry collision mesh filename=meshes/left_wrist_roll_rubber_hand.STL; visual mesh filename=meshes/left_wrist_roll_rubber_hand.STL
- link logo_link: geometry collision mesh filename=meshes/logo_link.STL; visual mesh filename=meshes/logo_link.STL
- link pelvis: geometry visual mesh filename=meshes/pelvis.STL
- link pelvis_contour_link: geometry collision mesh filename=meshes/pelvis_contour_link.STL; visual mesh filename=meshes/pelvis_contour_link.STL
- link right_ankle_pitch_link: geometry collision mesh filename=meshes/right_ankle_pitch_link.STL; visual mesh filename=meshes/right_ankle_pitch_link.STL
- link right_ankle_roll_link: geometry collision sphere radius=0.005; collision sphere radius=0.005
- link right_elbow_link: geometry collision mesh filename=meshes/right_elbow_link.STL; visual mesh filename=meshes/right_elbow_link.STL
- link right_hip_pitch_link: geometry collision mesh filename=meshes/right_hip_pitch_link.STL; visual mesh filename=meshes/right_hip_pitch_link.STL
- link right_hip_roll_link: geometry collision mesh filename=meshes/right_hip_roll_link.STL; visual mesh filename=meshes/right_hip_roll_link.STL
- link right_hip_yaw_link: geometry collision mesh filename=meshes/right_hip_yaw_link.STL; visual mesh filename=meshes/right_hip_yaw_link.STL
- link right_knee_link: geometry collision mesh filename=meshes/right_knee_link.STL; visual mesh filename=meshes/right_knee_link.STL
- link right_shoulder_pitch_link: geometry collision cylinder length=0.05 radius=0.03; visual mesh filename=meshes/right_shoulder_pitch_link.STL
- link right_shoulder_roll_link: geometry collision cylinder length=0.03 radius=0.03; visual mesh filename=meshes/right_shoulder_roll_link.STL
- link right_shoulder_yaw_link: geometry collision mesh filename=meshes/right_shoulder_yaw_link.STL; visual mesh filename=meshes/right_shoulder_yaw_link.STL
- link right_wrist_roll_rubber_hand: geometry collision mesh filename=meshes/right_wrist_roll_rubber_hand.STL; visual mesh filename=meshes/right_wrist_roll_rubber_hand.STL
- link torso_link: geometry collision mesh filename=meshes/torso_link_23dof_rev_1_0.STL; visual mesh filename=meshes/torso_link_23dof_rev_1_0.STL
Joints:
- removed joint floating_base
- joint left_ankle_pitch_joint: limit lower=-0.87267 upper=0.5236 effort=50 velocity=37 -> lower=-0.87267 upper=0.5236 effort=35 velocity=30
- joint left_ankle_roll_joint: limit lower=-0.2618 upper=0.2618 effort=50 velocity=37 -> lower=-0.2618 upper=0.2618 effort=35 velocity=30
- joint right_ankle_pitch_joint: limit lower=-0.87267 upper=0.5236 effort=50 velocity=37 -> lower=-0.87267 upper=0.5236 effort=35 velocity=30
- joint right_ankle_roll_joint: limit lower=-0.2618 upper=0.2618 effort=50 velocity=37 -> lower=-0.2618 upper=0.2618 effort=35 velocity=30
