Commit message: fix: update inertia of g1_29dof_rev_1_0.urdf

File: src/robots/g1_description/urdf/g1_29dof_rev_1_0_modify_inertia.urdf (robot description, URDF)
Before this commit: robot g1_12dof, 32 links, 31 joints
Links:
- removed link left_wrist_roll_rubber_hand
- removed link right_wrist_roll_rubber_hand
- added link left_rubber_hand, mass 0.170; visual mesh filename=package://g1_description/meshes/left_rubber_hand.STL
- added link left_wrist_pitch_link, mass 0.48404956; collision mesh filename=package://g1_description/meshes/left_wrist_pitch_link.STL; visual mesh filename=package://g1_description/meshes/left_wrist_pitch_link.STL
- added link left_wrist_roll_link, mass 0.08544498; collision mesh filename=package://g1_description/meshes/left_wrist_roll_link.STL; visual mesh filename=package://g1_description/meshes/left_wrist_roll_link.STL
- added link left_wrist_yaw_link, mass 0.08457647; collision mesh filename=package://g1_description/meshes/left_wrist_yaw_link.STL; visual mesh filename=package://g1_description/meshes/left_wrist_yaw_link.STL
- added link right_rubber_hand, mass 0.170; visual mesh filename=package://g1_description/meshes/right_rubber_hand.STL
- added link right_wrist_pitch_link, mass 0.48404956; collision mesh filename=package://g1_description/meshes/right_wrist_pitch_link.STL; visual mesh filename=package://g1_description/meshes/right_wrist_pitch_link.STL
- added link right_wrist_roll_link, mass 0.08544498; collision mesh filename=package://g1_description/meshes/right_wrist_roll_link.STL; visual mesh filename=package://g1_description/meshes/right_wrist_roll_link.STL
- added link right_wrist_yaw_link, mass 0.08457647; collision mesh filename=package://g1_description/meshes/right_wrist_yaw_link.STL; visual mesh filename=package://g1_description/meshes/right_wrist_yaw_link.STL
- added link waist_roll_link, mass 0.086; visual mesh filename=package://g1_description/meshes/waist_roll_link_rev_1_0.STL
- added link waist_yaw_link, mass 0.214; visual mesh filename=package://g1_description/meshes/waist_yaw_link_rev_1_0.STL
- link torso_link: geometry collision mesh filename=package://g1_description/meshes/torso_link_rev_1_0.STL; visual mesh filename=package://g1_description/meshes/torso_link_rev_1_0.STL
Joints:
- added joint left_hand_palm_joint: type fixed, parent left_wrist_yaw_link, child left_rubber_hand, origin xyz=0.0415 0.003 0 rpy=0 0 0
- added joint left_wrist_pitch_joint: type revolute, parent left_wrist_roll_link, child left_wrist_pitch_link, origin xyz=0.038 0 0 rpy=0 0 0, axis 0 1 0, limit lower=-1.614429558 upper=1.614429558 effort=5 velocity=22
- added joint left_wrist_yaw_joint: type revolute, parent left_wrist_pitch_link, child left_wrist_yaw_link, origin xyz=0.046 0 0 rpy=0 0 0, axis 0 0 1, limit lower=-1.614429558 upper=1.614429558 effort=5 velocity=22
- added joint right_hand_palm_joint: type fixed, parent right_wrist_yaw_link, child right_rubber_hand, origin xyz=0.0415 -0.003 0 rpy=0 0 0
- added joint right_wrist_pitch_joint: type revolute, parent right_wrist_roll_link, child right_wrist_pitch_link, origin xyz=0.038 0 0 rpy=0 0 0, axis 0 1 0, limit lower=-1.614429558 upper=1.614429558 effort=5 velocity=22
- added joint right_wrist_yaw_joint: type revolute, parent right_wrist_pitch_link, child right_wrist_yaw_link, origin xyz=0.046 0 0 rpy=0 0 0, axis 0 0 1, limit lower=-1.614429558 upper=1.614429558 effort=5 velocity=22
- added joint waist_pitch_joint: type revolute, parent waist_roll_link, child torso_link, origin xyz=0 0 0 rpy=0 0 0, axis 0 1 0, limit lower=-0.52 upper=0.52 effort=35 velocity=30
- added joint waist_roll_joint: type revolute, parent waist_yaw_link, child waist_roll_link, origin xyz=-0.0039635 0 0.044 rpy=0 0 0, axis 1 0 0, limit lower=-0.52 upper=0.52 effort=35 velocity=30
- joint left_ankle_pitch_joint: limit lower=-0.87267 upper=0.5236 effort=50 velocity=37 -> lower=-0.87267 upper=0.5236 effort=35 velocity=30
- joint left_ankle_roll_joint: limit lower=-0.2618 upper=0.2618 effort=50 velocity=37 -> lower=-0.2618 upper=0.2618 effort=35 velocity=30
- joint left_elbow_joint: type fixed -> revolute
- joint left_shoulder_pitch_joint: type fixed -> revolute
- joint left_shoulder_roll_joint: type fixed -> revolute
- joint left_shoulder_yaw_joint: type fixed -> revolute
- joint left_wrist_roll_joint: child left_wrist_roll_rubber_hand -> left_wrist_roll_link; type fixed -> revolute
- joint right_ankle_pitch_joint: limit lower=-0.87267 upper=0.5236 effort=50 velocity=37 -> lower=-0.87267 upper=0.5236 effort=35 velocity=30
- joint right_ankle_roll_joint: limit lower=-0.2618 upper=0.2618 effort=50 velocity=37 -> lower=-0.2618 upper=0.2618 effort=35 velocity=30
- joint right_elbow_joint: type fixed -> revolute
- joint right_shoulder_pitch_joint: type fixed -> revolute
- joint right_shoulder_roll_joint: type fixed -> revolute
- joint right_shoulder_yaw_joint: type fixed -> revolute
- joint right_wrist_roll_joint: child right_wrist_roll_rubber_hand -> right_wrist_roll_link; type fixed -> revolute
- joint waist_yaw_joint: child torso_link -> waist_yaw_link; origin xyz=-0.0039635 0 0.044 rpy=0 0 0 -> xyz=0 0 0 rpy=0 0 0; type fixed -> revolute
