Commit message: v3.0.0 (#74)
# Release Notes

## 🚀 New Features 

### Merge ROS and ROS2

- Added a one-click build script `build.sh`, which automatically detects the system architecture and ROS version to select the appropriate compiler. If build artifacts from different versions exist, the script prompts the user whether to clean them automatically.

  ````bash
  Usage: ./build.sh [OPTIONS] [PACKAGE_NAMES...]
  
  Options:
    -c, --clean    Clean workspace (remove symlinks and build artifacts)
    -m, --cmake    Build using CMake (for hardware deployment only)
    -h, --help     Show this help message
  
  Examples:
    ./build.sh                    # Build all ROS packages
    ./build.sh package1 package2  # Build specific ROS packages
    ./build.sh -c                 # Clean all symlinks and build artifacts
    ./build.sh --clean package1   # Clean specific package and build artifacts
    ./build.sh -m                 # Build with CMake for hardware deployment
  ````

- Each package contains both `package.ros1.xml` and `package.ros2.xml`. The build script automatically links the appropriate version for compilation.

- The ROS version is passed into `CMakeLists.txt` via an environment variable, and conditional compilation is done using macros in the code.

- Unified `gazebo.launch`/`gazebo.launch.py` files. You can launch any robot by simply passing `rname`, and delete `default_rl_config` in cpp code and `cfg` in launch configs.

  ```bash
  # ROS1
  source devel/setup.bash
  roslaunch rl_sar gazebo.launch rname:=<ROBOT>
  
  # ROS2
  source install/setup.bash
  ros2 launch rl_sar gazebo.launch.py rname:=<ROBOT>
  ```

- Launching `controller_manager` is no longer included in the launch files. Instead, it is dynamically started as a process in the code. For ROS2, `joint_names` are read from `config.yaml` to determine joint order and are written to a temporary file for use by `robot_joint_controller`.

### FSM Refactor

- Decoupled `rl_sdk` from the FSM and added `FSMFactory`. Each robot now maintains its own independent `fsm.hpp` inside its `policy` folder, with a unique namespace and `RLFSMState`. Outside the namespace, `FSMFactory` is inherited, and all `RLFSMState`s are automatically registered to `FSMManager` using `REGISTER_FSM_FACTORY`. In `rl_sim/resl.cpp`, passing the robot name to `FSMManager` returns the corresponding FSM.

- Added a new interface `RequestStateChange(state_name)` for switching states, callable from higher layers.

- Navigation mode no longer requires a separate FSM or assigning a fixed policy. It can now be toggled via remote control or keyboard in any mode.

## 🔧 Control

- Replace `RLFSMStateWaiting` with `RLFSMStatePassive`, set kp=0, kd=8 as default.

- Unified keyboard and joystick control

  |Gamepad Control|Keyboard Control|Description|
  |---|---|---|
  |**Basic**|||
  |A|Num0|Move the robot from its initial program pose to the `default_dof_pos` defined in `base.yaml` using position control interpolation|
  |B|Num9|Move the robot from its current position to the initial program pose using position control interpolation|
  |X|N|Toggle navigation mode (disables velocity commands, receives `cmd_vel` topic)|
  |Y|N/A|N/A|
  |**Simulation**|||
  |RB+Y|R|Reset Gazebo environment (stand up fallen robot)|
  |RB+X|Enter|Toggle Gazebo run/stop (default: running state)|
  |**Motor**|||
  |LB+A|M|N/A (Recommended for motor enable)|
  |LB+B|K|N/A (Recommended for motor disable)|
  |LB+X|P|N/A Motor passive mode (`kp=0, kd=8`)|
  |LB+RB|N/A|N/A (Recommended for emergency stop)|
  |**Skill**|||
  |RB+DPadUp|Num1|Basic Locomotion|
  |RB+DPadDown|Num2|Skill 2|
  |RB+DPadLeft|Num3|Skill 3|
  |RB+DPadRight|Num4|Skill 4|
  |LB+DPadUp|Num5|Skill 5|
  |LB+DPadDown|Num6|Skill 6|
  |LB+DPadLeft|Num7|Skill 7|
  |LB+DPadRight|Num8|Skill 8|
  |**Movement**|||
  |LY Axis|W/S|Forward/Backward movement (X-axis)|
  |LX Axis|A/D|Left/Right movement (Y-axis)|
  |RX Axis|Q/E|Yaw rotation|
  |N/A (Release joystick)|Space|Reset all control commands to zero|

## 🔧 Improvements

- Renamed the `models` folder to `policy`.

- Updated version number to `x.x.x`

## 🤖 Support List

|Robot Name (rname:=)|Pre-Trained Policy|Real|
|-|-|-|
|Unitree-A1 (a1)|legged_gym (IsaacGym)|✅|
|Unitree-Go2 (go2)|himloco (IsaacGym)</br>robot_lab (IsaacSim)|✅</br>✅|
|Unitree-Go2W (go2w)|robot_lab (IsaacSim)|✅|
|Unitree-B2 (b2)|robot_lab (IsaacSim)|⚪|
|Unitree-B2W (b2w)|robot_lab (IsaacSim)|⚪|
|Unitree-G1 (g1)|unitree_rl_gym (IsaacGym)</br>robomimic pre-loco (IsaacGym)</br>robomimic_dance (IsaacGym)</br>robomimic_kick (IsaacGym)</br>robomimic_kungfu (IsaacGym)|✅</br>✅</br>✅</br>🚫</br>🚫|
|FFTAI-GR1T1 (gr1t1)|legged_gym (IsaacGym)|⚪|
|FFTAI-GR1T2 (gr1t2)|legged_gym (IsaacGym)|⚪|
|GoldenRetriever-L4W4 (l4w4)|legged_gym (IsaacGym)</br>robot_lab (IsaacSim)|✅</br>✅|

## 📦 How To Add Your Robot

The following uses `<ROBOT>/<CONFIG>` to represent your robot environment, with all paths relative to `rl_sar/src/`. You only need to create or modify the following files, and the names must exactly match those shown below. (You can refer to the corresponding files in `go2w` as examples.)

```yaml
# your robot description
robots/<ROBOT>_description/CMakeLists.txt
robots/<ROBOT>_description/package.ros1.xml
robots/<ROBOT>_description/package.ros2.xml
robots/<ROBOT>_description/xacro/robot.xacro
robots/<ROBOT>_description/xacro/gazebo.xacro
robots/<ROBOT>_description/config/robot_control.yaml
robots/<ROBOT>_description/config/robot_control_ros2.yaml

# your policy
rl_sar/policy/fsm.hpp
rl_sar/policy/<ROBOT>/fsm.hpp
rl_sar/policy/<ROBOT>/base.yaml  # This file must follow the physical robot's joint order
rl_sar/policy/<ROBOT>/<CONFIG>/config.yaml  # This file can use the joint order specified during training
rl_sar/policy/<ROBOT>/<CONFIG>/<POLICY>.pt  # Must be exported as JIT to be usable

# your real robot code
rl_sar/src/rl_real_<ROBOT>.cpp  # You can customize the forward() function as needed to adapt to your policy
```

## 🧠 Next Version Update:

- Standardize controller button mappings  
- Combine `state_mapping` and `command_mapping` to `joint_mapping`
- Update Unitree-Go2W policy  
- Update Unitree-G1 dance animations  

## ⚠️ Known issue:
- `ObservationBuffer` calculates `num_obs_total` using `num_obs * observations_history.size()`. This works when indexing values smaller than the array length (e.g., [0, 1, 2, 3] where all values < 4 or [0, 0, 0,1, 2, 3] where all values < 6). However, when the array contains values larger than its length (e.g., [20, 20, 20] where 20 > 3), indexing will fail since it exceeds the buffer's capacity.
- G1 may fall while performing dance movements
- The Python versions are no longer actively maintained. Community contributions are welcome!


Thanks for your support! 🚀  

**Full Changelog:** https://github.com/fan-ziqi/rl_sar/compare/v2.5...v3.0.0

File: src/robots/go2_description/xacro/gazebo.xacro (robot description, xacro)
@@ -1,4 +1,6 @@
 <?xml version="1.0"?>
-<robot>
+<robot xmlns:xacro="http://www.ros.org/wiki/xacro">
+    <xacro:property name="ros_version" value="$(env ROS_VERSION)" />
+    <xacro:if value="${int(ros_version) == 1}">
     <!-- ros_control plugin -->
     <gazebo>
@@ -120,4 +122,105 @@
         </visual>
     </gazebo>
+    </xacro:if>
+    <xacro:if value="${int(ros_version) == 2}">
+    <gazebo reference="imu_link">
+      <sensor name="imu_sensor" type="imu">
+      <plugin filename="libgazebo_ros_imu_sensor.so" name="imu_plugin">
+          <ros>
+            <namespace>/</namespace>
+            <remapping>~/out:=imu</remapping>
+          </ros>
+          <initial_orientation_as_reference>false</initial_orientation_as_reference>
+        </plugin>
+        <always_on>true</always_on>
+        <update_rate>100</update_rate>
+        <visualize>true</visualize>
+        <imu>
+          <angular_velocity>
+            <x>
+              <noise type="gaussian">
+                <mean>0.0</mean>
+                <stddev>2e-4</stddev>
+                <bias_mean>0.0000075</bias_mean>
+                <bias_stddev>0.0000008</bias_stddev>
+              </noise>
+            </x>
+            <y>
+              <noise type="gaussian">
+                <mean>0.0</mean>
+                <stddev>2e-4</stddev>
+                <bias_mean>0.0000075</bias_mean>
+                <bias_stddev>0.0000008</bias_stddev>
+              </noise>
+            </y>
+            <z>
+              <noise type="gaussian">
+                <mean>0.0</mean>
+                <stddev>2e-4</stddev>
+                <bias_mean>0.0000075</bias_mean>
+                <bias_stddev>0.0000008</bias_stddev>
+              </noise>
+            </z>
+          </angular_velocity>
+          <linear_acceleration>
+            <x>
+              <noise type="gaussian">
+                <mean>0.0</mean>
+                <stddev>1.7e-2</stddev>
+                <bias_mean>0.1</bias_mean>
+                <bias_stddev>0.001</bias_stddev>
+              </noise>
+            </x>
+            <y>
+              <noise type="gaussian">
+                <mean>0.0</mean>
+                <stddev>1.7e-2</stddev>
+                <bias_mean>0.1</bias_mean>
+                <bias_stddev>0.001</bias_stddev>
+              </noise>
+            </y>
+            <z>
+              <noise type="gaussian">
+                <mean>0.0</mean>
+                <stddev>1.7e-2</stddev>
+                <bias_mean>0.1</bias_mean>
+                <bias_stddev>0.001</bias_stddev>
+              </noise>
+            </z>
+          </linear_acceleration>
+        </imu>
+      </sensor>
+    </gazebo>
+    <ros2_control name="GazeboSystem" type="system">
+        <hardware>
+            <plugin>gazebo_ros2_control/GazeboSystem</plugin>
+        </hardware>
+        <xacro:macro name="joint_interface" params="joint_name torque_limit">
+            <joint name="${joint_name}">
+            <command_interface name="effort">
+                <param name="min">-${torque_limit}</param>
+                <param name="max">${torque_limit}</param>
+            </command_interface>
+            <state_interface name="position"/>
+            <state_interface name="velocity"/>
+            <state_interface name="effort"/>
+            </joint>
+        </xacro:macro>
+        <xacro:macro name="leg_joints" params="prefix">
+            <xacro:joint_interface joint_name="${prefix}_hip_joint" torque_limit="${hip_torque_max}"/>
+            <xacro:joint_interface joint_name="${prefix}_thigh_joint" torque_limit="${thigh_torque_max}"/>
+            <xacro:joint_interface joint_name="${prefix}_calf_joint" torque_limit="${calf_torque_max}"/>
+        </xacro:macro>
+        <xacro:leg_joints prefix="FR"/>
+        <xacro:leg_joints prefix="FL"/>
+        <xacro:leg_joints prefix="RR"/>
+        <xacro:leg_joints prefix="RL"/>
+    </ros2_control>
+    <gazebo>
+        <plugin name="gazebo_ros2_control" filename="libgazebo_ros2_control.so">
+            <parameters>$(find go2_description)/config/robot_control_ros2.yaml</parameters>
+        </plugin>
+    </gazebo>
+    </xacro:if>
     <gazebo reference="base">
         <turnGravityOff>false</turnGravityOff>

File: src/robots/go2w_description/urdf/go2w_description.urdf (robot description, URDF)
Before this commit: robot go2w_description, 34 links, 33 joints
Links:
- link FL_calf: geometry collision cylinder length=0.12 radius=0.012; visual mesh filename=package://go2w_description/meshes/calf.dae
- link FL_foot: geometry collision cylinder length=0.045 radius=0.086; visual mesh filename=package://go2w_description/meshes/left_wheel.dae
- link FL_hip: geometry collision cylinder length=0.04 radius=0.046; visual mesh filename=package://go2w_description/meshes/hip.dae
- link FL_thigh: geometry collision box size=0.11 0.0245 0.034; visual mesh filename=package://go2w_description/meshes/thigh.dae
- link FR_calf: geometry collision cylinder length=0.12 radius=0.013; visual mesh filename=package://go2w_description/meshes/calf_mirror.dae
- link FR_foot: geometry collision cylinder length=0.045 radius=0.086; visual mesh filename=package://go2w_description/meshes/right_wheel.dae
- link FR_hip: geometry collision cylinder length=0.04 radius=0.046; visual mesh filename=package://go2w_description/meshes/hip.dae
- link FR_thigh: geometry collision box size=0.11 0.0245 0.034; visual mesh filename=package://go2w_description/meshes/thigh_mirror.dae
- link RL_calf: geometry collision cylinder length=0.12 radius=0.013; visual mesh filename=package://go2w_description/meshes/calf.dae
- link RL_foot: geometry collision cylinder length=0.045 radius=0.086; visual mesh filename=package://go2w_description/meshes/left_wheel.dae
- link RL_hip: geometry collision cylinder length=0.04 radius=0.046; visual mesh filename=package://go2w_description/meshes/hip.dae
- link RL_thigh: geometry collision box size=0.11 0.0245 0.034; visual mesh filename=package://go2w_description/meshes/thigh.dae
- link RR_calf: geometry collision cylinder length=0.12 radius=0.013; visual mesh filename=package://go2w_description/meshes/calf_mirror.dae
- link RR_foot: geometry collision cylinder length=0.045 radius=0.086; visual mesh filename=package://go2w_description/meshes/right_wheel.dae
- link RR_hip: geometry collision cylinder length=0.04 radius=0.046; visual mesh filename=package://go2w_description/meshes/hip.dae
- link RR_thigh: geometry collision box size=0.11 0.0245 0.034; visual mesh filename=package://go2w_description/meshes/thigh_mirror.dae
- link trunk: geometry collision box size=0.3762 0.0935 0.114; visual mesh filename=package://go2w_description/meshes/base.dae

File: src/robots/gr1t2_description/urdf/GR1T2_simple.urdf (robot description, URDF)
Before this commit: robot GR1T2Simple, 36 links, 35 joints
Links:
- removed link z_link_imu
- added link imu_link; visual box size=0.05 0.05 0.02
Joints:
- joint z_joint_imu: child z_link_imu -> imu_link
