Commit message: fix: change all xacro to urdf

File: src/robots/a1_description/xacro/gazebo.xacro (robot description, xacro)
@@ -1,4 +1,7 @@
 <?xml version="1.0"?>
 <robot xmlns:xacro="http://www.ros.org/wiki/xacro">
+    <xacro:property name="hip_torque_max" value="33.5"/>
+    <xacro:property name="thigh_torque_max" value="33.5"/>
+    <xacro:property name="calf_torque_max" value="33.5"/>
     <xacro:property name="ros_version" value="$(env ROS_VERSION)" />
     <xacro:if value="${int(ros_version) == 1}">

File: src/robots/a1_description/xacro/robot.xacro (robot description, xacro)
@@ -1,125 +1,5 @@
 <?xml version="1.0"?>
-<robot name="a1" xmlns:xacro="http://www.ros.org/wiki/xacro">
-    <xacro:arg name="DEBUG" default="false"/>
-    <xacro:include filename="$(find a1_description)/xacro/const.xacro"/>
-    <xacro:include filename="$(find a1_description)/xacro/materials.xacro"/>
-    <xacro:include filename="$(find a1_description)/xacro/leg.xacro"/>
-    <xacro:include filename="$(find a1_description)/xacro/stairs.xacro"/>
+<robot name="a1_description" xmlns:xacro="http://www.ros.org/wiki/xacro">
+    <xacro:include filename="$(find a1_description)/urdf/a1_description.urdf"/>
     <xacro:include filename="$(find a1_description)/xacro/gazebo.xacro"/>
-    <!-- <xacro:include filename="$(find a1_gazebo)/launch/stairs.urdf.xacro"/> -->
-    <!-- <xacro:stairs stairs="15" xpos="0" ypos="0" zpos="0" /> -->
-    <!-- Rollover Protection mode will add an additional stick on the top, use "true" or "false" to switch it. -->
-    <xacro:property name="rolloverProtection" value="false"/>
-    <!-- Debug mode will hung up the robot, use "true" or "false" to switch it. -->
-    <xacro:if value="$(arg DEBUG)">
-        <link name="world"/>
-        <joint name="base_static_joint" type="fixed">
-            <origin rpy="0 0 0" xyz="0 0 0"/>
-            <parent link="world"/>
-            <child link="base"/>
-        </joint>
-    </xacro:if>
-    <link name="base">
-        <visual>
-            <origin rpy="0 0 0" xyz="0 0 0"/>
-            <geometry>
-                <box size="0.001 0.001 0.001"/>
-            </geometry>
-        </visual>
-    </link>
-    <joint name="floating_base" type="fixed">
-        <origin rpy="0 0 0" xyz="0 0 0"/>
-        <parent link="base"/>
-        <child link="trunk"/>
-    </joint>
-    <link name="trunk">
-        <visual>
-            <origin rpy="0 0 0" xyz="0 0 0"/>
-            <geometry>
-                <mesh filename="package://a1_description/meshes/trunk.dae" scale="1 1 1"/>
-            </geometry>
-            <material name="orange"/>
-        </visual>
-        <collision>
-            <origin rpy="0 0 0" xyz="0 0 0"/>
-            <geometry>
-                <box size="${trunk_length} ${trunk_width} ${trunk_height}"/>
-            </geometry>
-        </collision>
-        <inertial>
-            <origin rpy="0 0 0" xyz="${trunk_com_x} ${trunk_com_y} ${trunk_com_z}"/>
-            <mass value="${trunk_mass}"/>
-            <inertia
-                ixx="${trunk_ixx}" ixy="${trunk_ixy}" ixz="${trunk_ixz}"
-                iyy="${trunk_iyy}" iyz="${trunk_iyz}"
-                izz="${trunk_izz}"/>
-        </inertial>
-    </link>
-    <xacro:if value="${(rolloverProtection == 'true')}">
-        <joint name="stick_joint" type="fixed">
-            <parent link="trunk"/>
-            <child link="stick_link"/>
-            <origin rpy="0 0 0" xyz="${0.18} 0 ${stick_length/2.0+0.08}"/>
-        </joint>
-        <link name="stick_link">
-            <visual>
-                <geometry>
-                    <cylinder length="${stick_length}" radius="${stick_radius}"/>
-                </geometry>
-                <origin rpy="0 0 0" xyz="0 0 0"/>
-                <material name="white"/>
-            </visual>
-            <collision>
-                <geometry>
-                    <cylinder length="${stick_length}" radius="${stick_radius}"/>
-                </geometry>
-                <origin rpy="0 0 0" xyz="0 0 0"/>
-            </collision>
-            <inertial>
-                <mass value="${stick_mass}"/>
-                <inertia
-                    ixx="${stick_mass / 2.0 * (stick_radius*stick_radius)}" ixy="0.0" ixz="0.0"
-                    iyy="${stick_mass / 12.0 * (3*stick_radius*stick_radius + stick_length*stick_length)}" iyz="0.0"
-                    izz="${stick_mass / 12.0 * (3*stick_radius*stick_radius + stick_length*stick_length)}"/>
-            </inertial>
-        </link>
-    </xacro:if>
-    <joint name="imu_joint" type="fixed">
-        <parent link="trunk"/>
-        <child link="imu_link"/>
-        <origin rpy="0 0 0" xyz="0 0 0"/>
-    </joint>
-    <link name="imu_link">
-        <inertial>
-            <mass value="0.001"/>
-            <origin rpy="0 0 0" xyz="0 0 0"/>
-            <inertia ixx="0.0001" ixy="0" ixz="0" iyy="0.0001" iyz="0" izz="0.0001"/>
-        </inertial>
-        <visual>
-            <origin rpy="0 0 0" xyz="0 0 0"/>
-            <geometry>
-                <box size="0.001 0.001 0.001"/>
-            </geometry>
-            <material name="red"/>
-        </visual>
-        <collision>
-            <origin rpy="0 0 0" xyz="0 0 0"/>
-            <geometry>
-                <box size=".001 .001 .001"/>
-            </geometry>
-        </collision>
-    </link>
-    <xacro:leg name="FR" mirror="-1" mirror_dae="False" front_hind="1" front_hind_dae="True">
-        <origin rpy="0 0 0" xyz="${leg_offset_x} ${-leg_offset_y} 0"/>
-    </xacro:leg>
-    <xacro:leg name="FL" mirror="1" mirror_dae="True" front_hind="1" front_hind_dae="True">
-        <origin rpy="0 0 0" xyz="${leg_offset_x} ${leg_offset_y} 0"/>
-    </xacro:leg>
-    <xacro:leg name="RR" mirror="-1" mirror_dae="False" front_hind="-1" front_hind_dae="False">
-        <origin rpy="0 0 0" xyz="${-leg_offset_x} ${-leg_offset_y} 0"/>
-    </xacro:leg>
-    <xacro:leg name="RL" mirror="1" mirror_dae="True" front_hind="-1" front_hind_dae="False">
-        <origin rpy="0 0 0" xyz="${-leg_offset_x} ${leg_offset_y} 0"/>
-    </xacro:leg>
-    <!-- <xacro:stairs stairs="15" xpos="0" ypos="2.0" zpos="0" /> -->
 </robot>

File: src/robots/b2_description/xacro/gazebo.xacro (robot description, xacro)
@@ -1,4 +1,7 @@
 <?xml version="1.0"?>
 <robot xmlns:xacro="http://www.ros.org/wiki/xacro">
+    <xacro:property name="hip_torque_max" value="200"/>
+    <xacro:property name="thigh_torque_max" value="200"/>
+    <xacro:property name="calf_torque_max" value="320"/>
     <xacro:property name="ros_version" value="$(env ROS_VERSION)" />
     <xacro:if value="${int(ros_version) == 1}">

File: src/robots/b2_description/xacro/robot.xacro (robot description, xacro)
@@ -1,162 +1,5 @@
 <?xml version="1.0"?>
 <robot name="b2_description" xmlns:xacro="http://www.ros.org/wiki/xacro">
-    <xacro:include filename="$(find b2_description)/xacro/const.xacro"/>
-    <xacro:include filename="$(find b2_description)/xacro/materials.xacro"/>
-    <xacro:include filename="$(find b2_description)/xacro/leg.xacro"/>
+    <xacro:include filename="$(find b2_description)/urdf/b2_description.urdf"/>
     <xacro:include filename="$(find b2_description)/xacro/gazebo.xacro"/>
-    <!-- Rotor related joint and link is only for demonstrate location. -->
-    <!-- Actually, the rotor will rotate and the joint is not fixed. Reduction ratio should be considered. -->
-    <!-- Debug mode will hung up the robot, use "true" or "false" to switch it. -->
-    <xacro:if value="$(arg DEBUG)">
-        <link name="world"/>
-        <joint name="base_static_joint" type="fixed">
-            <origin rpy="0 0 0" xyz="0 0 0"/>
-            <parent link="world"/>
-            <child link="base"/>
-        </joint>
-    </xacro:if>
-    <link name="base">
-        <visual>
-            <origin rpy="0 0 0" xyz="0 0 0"/>
-            <geometry>
-                <box size="0.001 0.001 0.001"/>
-            </geometry>
-        </visual>
-    </link>
-    <joint name="floating_base" type="fixed">
-        <origin rpy="0 0 0" xyz="0 0 0"/>
-        <parent link="base"/>
-        <child link="trunk"/>
-    </joint>
-    <link name="trunk">
-        <visual>
-            <origin rpy="0 0 0" xyz="0 0 0"/>
-            <geometry>
-                <mesh filename="package://b2_description/meshes/trunk.dae" scale="1 1 1"/>
-            </geometry>
-            <!-- <material name="orange"/> -->
-        </visual>
-        <collision>
-            <origin rpy="0 0 0" xyz="0 0 0"/>
-            <geometry>
-                <box size="${trunk_length} ${trunk_width} ${trunk_height}"/>
-            </geometry>
-        </collision>
-        <!-- <collision>
-            <origin rpy="0 0 0" xyz="0 0 0"/>
-            <geometry>
-                <mesh filename="package://b1_description/meshes/trunk.dae" scale="1 1 1"/>
-            </geometry>
-        </collision> -->
-        <inertial>
-            <origin rpy="0 0 0" xyz="${trunk_com_x} ${trunk_com_y} ${trunk_com_z}"/>
-            <mass value="${trunk_mass}"/>
-            <inertia
-                ixx="${trunk_ixx}" ixy="${trunk_ixy}" ixz="${trunk_ixz}"
-                iyy="${trunk_iyy}" iyz="${trunk_iyz}"
-                izz="${trunk_izz}"/>
-        </inertial>
-    </link>
-    <joint name="imu_joint" type="fixed">
-        <parent link="trunk"/>
-        <child link="imu_link"/>
-        <origin rpy="0 0 0" xyz="0 0 0"/>
-    </joint>
-    <link name="imu_link">
-        <inertial>
-            <mass value="0.001"/>
-            <origin rpy="0 0 0" xyz="0 0 0"/>
-            <inertia ixx="0.0001" ixy="0" ixz="0" iyy="0.0001" iyz="0" izz="0.0001"/>
-        </inertial>
-        <visual>
-            <origin rpy="0 0 0" xyz="0 0 0"/>
-            <geometry>
-                <box size="0.001 0.001 0.001"/>
-            </geometry>
-            <!-- <material name="red"/> -->
-        </visual>
-        <collision>
-            <origin rpy="0 0 0" xyz="0 0 0"/>
-            <geometry>
-                <box size=".001 .001 .001"/>
-            </geometry>
-        </collision>
-    </link>
-    <joint name="head_joint" type="fixed">
-        <parent link="trunk"/>
-        <child link="head_Link"/>
-        <origin rpy="0 0 0" xyz="0 0 0"/>
-    </joint>
-    <link name="head_Link">
-        <inertial>
-            <origin rpy="0 0 0" xyz="0.33989 -0.000168 0.12029"/>
-            <mass value="3.366" />
-            <inertia
-            ixx="0.026455"
-            ixy="3.15E-05"
-            ixz="0.00166"
-            iyy="0.029221"
-            iyz="-3.27E-05"
-            izz="0.010918" />
-        </inertial>
-        <collision>
-            <origin rpy="0 0 0" xyz="0.41 0 0.005"/>
-            <geometry>
-                <box size="0.04 0.12 0.14" />
-            </geometry>
-        </collision>
-    </link>
-    <joint name="lidar_joint" type="fixed">
-        <parent link="trunk"/>
-        <child link="lidar_link"/>
-        <origin rpy="0 0 0" xyz="0.34218 0 0.17851"/>
-    </joint>
-    <link name="lidar_link">
-        <inertial>
-            <origin rpy="0 0 0" xyz="0 0 0"/>
-            <mass value="6.55E-08" />
-            <inertia
-            ixx="1.64E-15"
-            ixy="0"
-            ixz="-1.09E-47"
-            iyy="1.64E-15"
-            iyz="-1.32E-47"
-            izz="1.64E-15" />
-        </inertial>
-        <collision>
-            <origin rpy="0 0 0" xyz="0 0 -0.02"/>
-            <geometry>
-                <cylinder length="0.16" radius="0.076" />
-            </geometry>
-        </collision>
-    </link>
-    <joint name="tail_joint" type="fixed">
-        <parent link="trunk"/>
-        <child link="tail_link"/>
-        <origin rpy="0 0 0" xyz="0 0 0"/>
-    </joint>
-    <link name="tail_link">
-        <inertial>
-            <origin rpy="0 0 0" xyz="-0.37448 0.000488 0.006495"/>
-            <mass value="0.777" />
-            <inertia
-            ixx="0.0028118"
-            ixy="1.95E-05"
-            ixz="-7.87E-06"
-            iyy="0.0047506"
-            iyz="-1.57E-05"
-            izz="0.0029154" />
-        </inertial>
-        <collision>
-            <origin rpy="0 0 0" xyz="-0.405 0 0.005"/>
-            <geometry>
-                <box size="0.025 0.12 0.14" />
-            </geometry>
-        </collision>
-    </link>
-    <xacro:leg name="FR" mirror="-1" mirror_dae= "False" front_hind="1"  front_hind_dae="True"  />
-    <xacro:leg name="FL" mirror="1"  mirror_dae="True"   front_hind="1"  front_hind_dae="True"  />
-    <xacro:leg name="RR" mirror="-1" mirror_dae="False"  front_hind="-1" front_hind_dae="False" />
-    <xacro:leg name="RL" mirror="1"  mirror_dae="True"   front_hind="-1" front_hind_dae="False" />
-    <!-- <xacro:stairs stairs="15" xpos="0" ypos="2.0" zpos="0" /> -->
 </robot>

File: src/robots/b2w_description/xacro/gazebo.xacro (robot description, xacro)
@@ -1,4 +1,7 @@
 <?xml version="1.0"?>
 <robot xmlns:xacro="http://www.ros.org/wiki/xacro">
+    <xacro:property name="hip_torque_max" value="200"/>
+    <xacro:property name="thigh_torque_max" value="200"/>
+    <xacro:property name="calf_torque_max" value="320"/>
     <xacro:property name="ros_version" value="$(env ROS_VERSION)" />
     <xacro:if value="${int(ros_version) == 1}">

File: src/robots/b2w_description/xacro/robot.xacro (robot description, xacro)
@@ -1,162 +1,5 @@
 <?xml version="1.0"?>
 <robot name="b2w_description" xmlns:xacro="http://www.ros.org/wiki/xacro">
-    <xacro:include filename="$(find b2w_description)/xacro/const.xacro"/>
-    <xacro:include filename="$(find b2w_description)/xacro/materials.xacro"/>
-    <xacro:include filename="$(find b2w_description)/xacro/leg.xacro"/>
+    <xacro:include filename="$(find b2w_description)/urdf/b2w_description.urdf"/>
     <xacro:include filename="$(find b2w_description)/xacro/gazebo.xacro"/>
-    <!-- Rotor related joint and link is only for demonstrate location. -->
-    <!-- Actually, the rotor will rotate and the joint is not fixed. Reduction ratio should be considered. -->
-    <!-- Debug mode will hung up the robot, use "true" or "false" to switch it. -->
-    <xacro:if value="$(arg DEBUG)">
-        <link name="world"/>
-        <joint name="base_static_joint" type="fixed">
-            <origin rpy="0 0 0" xyz="0 0 0"/>
-            <parent link="world"/>
-            <child link="base"/>
-        </joint>
-    </xacro:if>
-    <link name="base">
-        <visual>
-            <origin rpy="0 0 0" xyz="0 0 0"/>
-            <geometry>
-                <box size="0.001 0.001 0.001"/>
-            </geometry>
-        </visual>
-    </link>
-    <joint name="floating_base" type="fixed">
-        <origin rpy="0 0 0" xyz="0 0 0"/>
-        <parent link="base"/>
-        <child link="trunk"/>
-    </joint>
-    <link name="trunk">
-        <visual>
-            <origin rpy="0 0 0" xyz="0 0 0"/>
-            <geometry>
-                <mesh filename="package://b2w_description/meshes/trunk.dae" scale="1 1 1"/>
-            </geometry>
-            <!-- <material name="orange"/> -->
-        </visual>
-        <collision>
-            <origin rpy="0 0 0" xyz="0 0 0"/>
-            <geometry>
-                <box size="${trunk_length} ${trunk_width} ${trunk_height}"/>
-            </geometry>
-        </collision>
-        <!-- <collision>
-            <origin rpy="0 0 0" xyz="0 0 0"/>
-            <geometry>
-                <mesh filename="package://b1_description/meshes/trunk.dae" scale="1 1 1"/>
-            </geometry>
-        </collision> -->
-        <inertial>
-            <origin rpy="0 0 0" xyz="${trunk_com_x} ${trunk_com_y} ${trunk_com_z}"/>
-            <mass value="${trunk_mass}"/>
-            <inertia
-                ixx="${trunk_ixx}" ixy="${trunk_ixy}" ixz="${trunk_ixz}"
-                iyy="${trunk_iyy}" iyz="${trunk_iyz}"
-                izz="${trunk_izz}"/>
-        </inertial>
-    </link>
-    <joint name="imu_joint" type="fixed">
-        <parent link="trunk"/>
-        <child link="imu_link"/>
-        <origin rpy="0 0 0" xyz="0 0 0"/>
-    </joint>
-    <link name="imu_link">
-        <inertial>
-            <mass value="0.001"/>
-            <origin rpy="0 0 0" xyz="0 0 0"/>
-            <inertia ixx="0.0001" ixy="0" ixz="0" iyy="0.0001" iyz="0" izz="0.0001"/>
-        </inertial>
-        <visual>
-            <origin rpy="0 0 0" xyz="0 0 0"/>
-            <geometry>
-                <box size="0.001 0.001 0.001"/>
-            </geometry>
-            <!-- <material name="red"/> -->
-        </visual>
-        <collision>
-            <origin rpy="0 0 0" xyz="0 0 0"/>
-            <geometry>
-                <box size=".001 .001 .001"/>
-            </geometry>
-        </collision>
-    </link>
-    <joint name="head_joint" type="fixed">
-        <parent link="trunk"/>
-        <child link="head_Link"/>
-        <origin rpy="0 0 0" xyz="0 0 0"/>
-    </joint>
-    <link name="head_Link">
-        <inertial>
-            <origin rpy="0 0 0" xyz="0.33989 -0.000168 0.12029"/>
-            <mass value="3.366" />
-            <inertia
-            ixx="0.026455"
-            ixy="3.15E-05"
-            ixz="0.00166"
-            iyy="0.029221"
-            iyz="-3.27E-05"
-            izz="0.010918" />
-        </inertial>
-        <collision>
-            <origin rpy="0 0 0" xyz="0.41 0 0.005"/>
-            <geometry>
-                <box size="0.04 0.12 0.14" />
-            </geometry>
-        </collision>
-    </link>
-    <joint name="lidar_joint" type="fixed">
-        <parent link="trunk"/>
-        <child link="lidar_link"/>
-        <origin rpy="0 0 0" xyz="0.34218 0 0.17851"/>
-    </joint>
-    <link name="lidar_link">
-        <inertial>
-            <origin rpy="0 0 0" xyz="0 0 0"/>
-            <mass value="6.55E-08" />
-            <inertia
-            ixx="1.64E-15"
-            ixy="0"
-            ixz="-1.09E-47"
-            iyy="1.64E-15"
-            iyz="-1.32E-47"
-            izz="1.64E-15" />
-        </inertial>
-        <collision>
-            <origin rpy="0 0 0" xyz="0 0 -0.02"/>
-            <geometry>
-                <cylinder length="0.16" radius="0.076" />
-            </geometry>
-        </collision>
-    </link>
-    <joint name="tail_joint" type="fixed">
-        <parent link="trunk"/>
-        <child link="tail_link"/>
-        <origin rpy="0 0 0" xyz="0 0 0"/>
-    </joint>
-    <link name="tail_link">
-        <inertial>
-            <origin rpy="0 0 0" xyz="-0.37448 0.000488 0.006495"/>
-            <mass value="0.777" />
-            <inertia
-            ixx="0.0028118"
-            ixy="1.95E-05"
-            ixz="-7.87E-06"
-            iyy="0.0047506"
-            iyz="-1.57E-05"
-            izz="0.0029154" />
-        </inertial>
-        <collision>
-            <origin rpy="0 0 0" xyz="-0.405 0 0.005"/>
-            <geometry>
-                <box size="0.025 0.12 0.14" />
-            </geometry>
-        </collision>
-    </link>
-    <xacro:leg name="FR" mirror="-1" mirror_dae= "False" front_hind="1"  front_hind_dae="True"  />
-    <xacro:leg name="FL" mirror="1"  mirror_dae="True"   front_hind="1"  front_hind_dae="True"  />
-    <xacro:leg name="RR" mirror="-1" mirror_dae="False"  front_hind="-1" front_hind_dae="False" />
-    <xacro:leg name="RL" mirror="1"  mirror_dae="True"   front_hind="-1" front_hind_dae="False" />
-    <!-- <xacro:stairs stairs="15" xpos="0" ypos="2.0" zpos="0" /> -->
 </robot>

File: src/robots/go2_description/xacro/gazebo.xacro (robot description, xacro)
@@ -1,4 +1,7 @@
 <?xml version="1.0"?>
 <robot xmlns:xacro="http://www.ros.org/wiki/xacro">
+    <xacro:property name="hip_torque_max" value="23.7"/>
+    <xacro:property name="thigh_torque_max" value="23.7"/>
+    <xacro:property name="calf_torque_max" value="35.55"/>
     <xacro:property name="ros_version" value="$(env ROS_VERSION)" />
     <xacro:if value="${int(ros_version) == 1}">
