Commit message: fix: broken link of go2_description

File: src/robots/go2_description/urdf/go2_description.urdf (robot description, URDF)
Before this commit: robot go2_description, 29 links, 28 joints
Links:
- removed link imu
- added link imu_link, mass 0
- added link trunk, mass 6.921; collision box size=0.3762 0.0935 0.114; visual mesh filename=package://go2_description/meshes/base.dae
- link FL_calf: geometry collision cylinder length=0.12 radius=0.012; visual mesh filename=package://go2_description/meshes/calf.dae
- link FL_foot: geometry collision sphere radius=0.022; visual mesh filename=package://go2_description/meshes/foot.dae
- link FL_hip: geometry collision cylinder length=0.04 radius=0.046; visual mesh filename=package://go2_description/meshes/hip.dae
- link FL_thigh: geometry collision box size=0.213 0.0245 0.034; visual mesh filename=package://go2_description/meshes/thigh.dae
- link FR_calf: geometry collision cylinder length=0.12 radius=0.013; visual mesh filename=package://go2_description/meshes/calf_mirror.dae
- link FR_foot: geometry collision sphere radius=0.022; visual mesh filename=package://go2_description/meshes/foot.dae
- link FR_hip: geometry collision cylinder length=0.04 radius=0.046; visual mesh filename=package://go2_description/meshes/hip.dae
- link FR_thigh: geometry collision box size=0.213 0.0245 0.034; visual mesh filename=package://go2_description/meshes/thigh_mirror.dae
- link RL_calf: geometry collision cylinder length=0.12 radius=0.013; visual mesh filename=package://go2_description/meshes/calf.dae
- link RL_foot: geometry collision sphere radius=0.022; visual mesh filename=package://go2_description/meshes/foot.dae
- link RL_hip: geometry collision cylinder length=0.04 radius=0.046; visual mesh filename=package://go2_description/meshes/hip.dae
- link RL_thigh: geometry collision box size=0.213 0.0245 0.034; visual mesh filename=package://go2_description/meshes/thigh.dae
- link RR_calf: geometry collision cylinder length=0.12 radius=0.013; visual mesh filename=package://go2_description/meshes/calf_mirror.dae
- link RR_foot: geometry collision sphere radius=0.022; visual mesh filename=package://go2_description/meshes/foot.dae
- link RR_hip: geometry collision cylinder length=0.04 radius=0.046; visual mesh filename=package://go2_description/meshes/hip.dae
- link RR_thigh: geometry collision box size=0.213 0.0245 0.034; visual mesh filename=package://go2_description/meshes/thigh_mirror.dae
- link base: mass 6.921 -> None; geometry visual box size=0.001 0.001 0.001
Joints:
- added joint floating_base: type fixed, parent base, child trunk, origin xyz=0 0 0 rpy=0 0 0
- joint FL_hip_joint: parent base -> trunk
- joint FR_hip_joint: parent base -> trunk
- joint Head_upper_joint: parent base -> trunk
- joint RL_hip_joint: parent base -> trunk
- joint RR_hip_joint: parent base -> trunk
- joint imu_joint: child imu -> imu_link; parent base -> trunk
- joint radar_joint: parent base -> trunk
