Commit message: 0622

File: src/robots/go2w_description/urdf/go2w_description.urdf (robot description, URDF)
Before this commit: robot go2w_description, 34 links, 33 joints
Links:
- link FL_calf: geometry collision cylinder length=0.12 radius=0.012; visual mesh filename=package://go2w_description/meshes/calf.dae
- link FL_foot: geometry collision cylinder length=0.045 radius=0.086; visual mesh filename=package://go2w_description/meshes/left_wheel.dae
- link FL_hip: geometry collision cylinder length=0.04 radius=0.046; visual mesh filename=package://go2w_description/meshes/hip.dae
- link FL_thigh: geometry collision box size=0.11 0.0245 0.034; visual mesh filename=package://go2w_description/meshes/thigh.dae
- link FR_calf: geometry collision cylinder length=0.12 radius=0.013; visual mesh filename=package://go2w_description/meshes/calf_mirror.dae
- link FR_foot: geometry collision cylinder length=0.045 radius=0.086; visual mesh filename=package://go2w_description/meshes/right_wheel.dae
- link FR_hip: geometry collision cylinder length=0.04 radius=0.046; visual mesh filename=package://go2w_description/meshes/hip.dae
- link FR_thigh: geometry collision box size=0.11 0.0245 0.034; visual mesh filename=package://go2w_description/meshes/thigh_mirror.dae
- link RL_calf: geometry collision cylinder length=0.12 radius=0.013; visual mesh filename=package://go2w_description/meshes/calf.dae
- link RL_foot: geometry collision cylinder length=0.045 radius=0.086; visual mesh filename=package://go2w_description/meshes/left_wheel.dae
- link RL_hip: geometry collision cylinder length=0.04 radius=0.046; visual mesh filename=package://go2w_description/meshes/hip.dae
- link RL_thigh: geometry collision box size=0.11 0.0245 0.034; visual mesh filename=package://go2w_description/meshes/thigh.dae
- link RR_calf: geometry collision cylinder length=0.12 radius=0.013; visual mesh filename=package://go2w_description/meshes/calf_mirror.dae
- link RR_foot: geometry collision cylinder length=0.045 radius=0.086; visual mesh filename=package://go2w_description/meshes/right_wheel.dae
- link RR_hip: geometry collision cylinder length=0.04 radius=0.046; visual mesh filename=package://go2w_description/meshes/hip.dae
- link RR_thigh: geometry collision box size=0.11 0.0245 0.034; visual mesh filename=package://go2w_description/meshes/thigh_mirror.dae
- link trunk: geometry collision box size=0.3762 0.0935 0.114; visual mesh filename=package://go2w_description/meshes/base.dae

File: src/robots/go2w_description/xacro/robot.xacro (robot description, xacro)
@@ -1,5 +1,5 @@
 <?xml version="1.0"?>
 <robot name="go2w_description" xmlns:xacro="http://www.ros.org/wiki/xacro">
-    <xacro:include filename="$(find b2w_description)/urdf/go2w_description.urdf"/>
-    <xacro:include filename="$(find b2w_description)/xacro/gazebo.xacro"/>
+    <xacro:include filename="$(find go2w_description)/urdf/go2w_description.urdf"/>
+    <xacro:include filename="$(find go2w_description)/xacro/gazebo.xacro"/>
 </robot>

File: src/robots/gr1t1_description/xacro/robot.xacro (robot description, xacro)
@@ -1,5 +1,5 @@
 <?xml version="1.0"?>
-<robot name="go2w_description" xmlns:xacro="http://www.ros.org/wiki/xacro">
-    <xacro:include filename="$(find b2w_description)/urdf/go2w_description.urdf"/>
-    <xacro:include filename="$(find b2w_description)/xacro/gazebo.xacro"/>
+<robot name="gr1t1_description" xmlns:xacro="http://www.ros.org/wiki/xacro">
+    <xacro:include filename="$(find gr1t1_description)/urdf/GR1T1_lower_limb.urdf"/>
+    <xacro:include filename="$(find gr1t1_description)/xacro/gazebo.xacro"/>
 </robot>

File: src/robots/gr1t2_description/xacro/gazebo.xacro (robot description, xacro)
@@ -6,5 +6,5 @@
     <gazebo>
         <plugin filename="libgazebo_ros_control.so" name="gazebo_ros_control">
-        <robotNamespace>/gr1t1_gazebo</robotNamespace>
+        <robotNamespace>/gr1t2_gazebo</robotNamespace>
         <robotSimType>gazebo_ros_control/DefaultRobotHWSim</robotSimType>
         </plugin>

File: src/robots/l4w4_description/xacro/gazebo.xacro (robot description, xacro)
@@ -9,5 +9,5 @@
     <gazebo>
         <plugin name="gazebo_ros_control" filename="libgazebo_ros_control.so">
-            <robotNamespace>/go2w_gazebo</robotNamespace>
+            <robotNamespace>/l4w4_gazebo</robotNamespace>
             <robotSimType>gazebo_ros_control/DefaultRobotHWSim</robotSimType>
         </plugin>
@@ -347,5 +347,5 @@
     <gazebo>
         <plugin name="gazebo_ros2_control" filename="libgazebo_ros2_control.so">
-            <parameters>$(find go2w_description)/config/robot_control_ros2.yaml</parameters>
+            <parameters>$(find l4w4_description)/config/robot_control_ros2.yaml</parameters>
         </plugin>
     </gazebo>

Commit message: fix: update latest go2w_description.urdf

File: src/robots/go2w_description/urdf/go2w_description.urdf (robot description, URDF)
Before this commit: robot go2w_description, 34 links, 33 joints
Links:
- removed link radar
- added link radar_link, mass 0
- link FL_calf: geometry collision cylinder length=0.12 radius=0.012; visual mesh filename=package://go2w_description/meshes/calf.stl
- link FL_foot: geometry collision mesh filename=package://go2w_description/meshes/left_wheel.dae; visual mesh filename=package://go2w_description/meshes/left_wheel.dae
- link FR_calf: geometry collision cylinder length=0.12 radius=0.013; visual mesh filename=package://go2w_description/meshes/calf_mirror.stl
- link FR_foot: geometry collision mesh filename=package://go2w_description/meshes/right_wheel.dae; visual mesh filename=package://go2w_description/meshes/right_wheel.dae
- link RL_calf: geometry collision cylinder length=0.12 radius=0.013; visual mesh filename=package://go2w_description/meshes/calf.stl
- link RL_foot: geometry collision mesh filename=package://go2w_description/meshes/left_wheel.dae; visual mesh filename=package://go2w_description/meshes/left_wheel.dae
- link RR_calf: geometry collision cylinder length=0.12 radius=0.013; visual mesh filename=package://go2w_description/meshes/calf_mirror.stl
- link RR_foot: geometry collision mesh filename=package://go2w_description/meshes/right_wheel.dae; visual mesh filename=package://go2w_description/meshes/right_wheel.dae
Joints:
- joint FL_foot_joint: limit lower=-999999 upper=999999 effort=23.7 velocity=30.1 -> effort=23.7 velocity=30.1; type revolute -> continuous
- joint FR_foot_joint: limit lower=-999999 upper=999999 effort=23.7 velocity=30.1 -> effort=23.7 velocity=30.1; type revolute -> continuous
- joint RL_foot_joint: limit lower=-999999 upper=999999 effort=23.7 velocity=30.1 -> effort=23.7 velocity=30.1; type revolute -> continuous
- joint RR_foot_joint: limit lower=-999999 upper=999999 effort=23.7 velocity=30.1 -> effort=23.7 velocity=30.1; type revolute -> continuous
- joint radar_joint: child radar -> radar_link
