Commit message: change model

File: src/robots/lite3_description/urdf/Lite3.urdf (robot description, URDF)
Before this commit: robot Lite3, 19 links, 18 joints
Links:
- link FL_HIP: geometry visual mesh filename=package://lite3_description/meshes/FL_HIP.dae
- link FL_SHANK: geometry collision box size=0.02 0.02 0.18; visual mesh filename=package://lite3_description/meshes/SHANK.dae
- link FL_THIGH: geometry collision box size=0.02 0.02 0.16; visual mesh filename=package://lite3_description/meshes/L_THIGH.dae
- link FR_HIP: geometry visual mesh filename=package://lite3_description/meshes/FR_HIP.dae
- link FR_SHANK: geometry collision box size=0.02 0.02 0.18; visual mesh filename=package://lite3_description/meshes/SHANK.dae
- link FR_THIGH: geometry collision box size=0.02 0.02 0.16; visual mesh filename=package://lite3_description/meshes/R_THIGH.dae
- link HL_HIP: geometry visual mesh filename=package://lite3_description/meshes/HL_HIP.dae
- link HL_SHANK: geometry collision box size=0.02 0.02 0.18; visual mesh filename=package://lite3_description/meshes/SHANK.dae
- link HL_THIGH: geometry collision box size=0.02 0.02 0.16; visual mesh filename=package://lite3_description/meshes/L_THIGH.dae
- link HR_HIP: geometry visual mesh filename=package://lite3_description/meshes/HR_HIP.dae
- link HR_SHANK: geometry collision box size=0.02 0.02 0.18; visual mesh filename=package://lite3_description/meshes/SHANK.dae
- link HR_THIGH: geometry collision box size=0.02 0.02 0.16; visual mesh filename=package://lite3_description/meshes/R_THIGH.dae
- link TORSO: geometry collision box size=0.234 0.184 0.08; visual mesh filename=package://lite3_description/meshes/TORSO.dae

Commit message: change model

File: src/robots/lite3_description/urdf/Lite3.urdf (robot description, URDF)
Before this commit: robot Lite3, 19 links, 18 joints
Links:
- removed link radar
Joints:
- removed joint radar_joint
