Commit message: update

File: src/robots/lite3_description/urdf/lite3.urdf (robot description, URDF)
Before this commit: robot Lite3, 18 links, 17 joints
Links:
- added link base; visual box size=0.001 0.001 0.001
Joints:
- added joint floating_base: type fixed, parent base, child TORSO, origin xyz=0 0 0 rpy=0 0 0

File: src/robots/lite3_description/xacro/gazebo.xacro (robot description, xacro)
@@ -5,4 +5,126 @@
     <xacro:property name="Knee_torque_max" value="30"/>
     <xacro:property name="ros_version" value="$(env ROS_VERSION)" />
+    <xacro:if value="${int(ros_version) == 1}">
+    <!-- ros_control plugin -->
+    <gazebo>
+        <plugin name="gazebo_ros_control" filename="libgazebo_ros_control.so">
+            <robotNamespace>/lite3_gazebo</robotNamespace>
+            <robotSimType>gazebo_ros_control/DefaultRobotHWSim</robotSimType>
+        </plugin>
+    </gazebo>
+    <!-- Show the trajectory of TORSO center. -->
+    <!-- <gazebo>
+        <plugin name="3dplot" filename="libLinkPlot3DPlugin.so">
+            <frequency>10</frequency>
+            <plot>
+                <link>base</link>
+                <pose>0 0 0 0 0 0</pose>
+                <material>Gazebo/Yellow</material>
+            </plot>
+        </plugin>
+    </gazebo> -->
+    <!-- Show the trajectory of foot. You can add another trajectory about another foot. -->
+    <!-- <gazebo>
+        <plugin name="3dplot" filename="libLinkPlot3DPlugin.so">
+            <frequency>100</frequency>
+            <plot>
+                <link>FL_foot</link>
+                <pose>0 0 0 0 0 0</pose>
+                <material>Gazebo/Green</material>
+            </plot>
+        </plugin>
+    </gazebo> -->
+    <gazebo>
+        <plugin filename="libgazebo_ros_force.so" name="gazebo_ros_force">
+            <bodyName>TORSO</bodyName>
+            <topicName>/apply_force/TORSO</topicName>
+        </plugin>
+    </gazebo>
+    <gazebo reference="imu_link">
+        <gravity>true</gravity>
+        <sensor name="imu_sensor" type="imu">
+            <always_on>true</always_on>
+            <update_rate>1000</update_rate>
+            <visualize>true</visualize>
+            <topic>__default_topic__</topic>
+            <plugin filename="libgazebo_ros_imu_sensor.so" name="imu_plugin">
+                <topicName>TORSO_imu</topicName>
+                <bodyName>imu_link</bodyName>
+                <updateRateHZ>1000.0</updateRateHZ>
+                <gaussianNoise>0.0</gaussianNoise>
+                <xyzOffset>0 0 0</xyzOffset>
+                <rpyOffset>0 0 0</rpyOffset>
+                <frameName>imu_link</frameName>
+            </plugin>
+            <pose>0 0 0 0 0 0</pose>
+        </sensor>
+    </gazebo>
+    <!-- Foot contacts. -->
+    <gazebo reference="FR_calf">
+        <sensor name="FR_foot_contact" type="contact">
+        <update_rate>100</update_rate>
+        <plugin name="contactPlugin" filename="libunitreeFootContactPlugin.so"/>
+        <contact>
+            <collision>FR_calf_fixed_joint_lump__FR_foot_collision_1</collision>
+        </contact>
+        </sensor>
+    </gazebo>
+    <gazebo reference="FL_calf">
+        <sensor name="FL_foot_contact" type="contact">
+        <update_rate>100</update_rate>
+        <plugin name="contactPlugin" filename="libunitreeFootContactPlugin.so"/>
+        <contact>
+            <collision>FL_calf_fixed_joint_lump__FL_foot_collision_1</collision>
+        </contact>
+        </sensor>
+    </gazebo>
+    <gazebo reference="HR_calf">
+        <sensor name="HR_foot_contact" type="contact">
+        <update_rate>100</update_rate>
+        <plugin name="contactPlugin" filename="libunitreeFootContactPlugin.so"/>
+        <contact>
+            <collision>HR_calf_fixed_joint_lump__HR_foot_collision_1</collision>
+        </contact>
+        </sensor>
+    </gazebo>
+    <gazebo reference="HL_calf">
+        <sensor name="HL_foot_contact" type="contact">
+        <update_rate>100</update_rate>
+        <plugin name="contactPlugin" filename="libunitreeFootContactPlugin.so"/>
+        <contact>
+            <collision>HL_calf_fixed_joint_lump__HL_foot_collision_1</collision>
+        </contact>
+        </sensor>
+    </gazebo>
+    <!-- Visualization of Foot contacts. -->
+    <!-- <gazebo reference="FR_foot">
+        <visual>
+            <plugin name="drawForcePlugin" filename="libunitreeDrawForcePlugin.so">
+                <topicName>FR_foot_contact</topicName>
+            </plugin>
+        </visual>
+    </gazebo>
+    <gazebo reference="FL_foot">
+        <visual>
+            <plugin name="drawForcePlugin" filename="libunitreeDrawForcePlugin.so">
+                <topicName>FL_foot_contact</topicName>
+            </plugin>
+        </visual>
+    </gazebo>
+    <gazebo reference="HR_foot">
+        <visual>
+            <plugin name="drawForcePlugin" filename="libunitreeDrawForcePlugin.so">
+                <topicName>HR_foot_contact</topicName>
+            </plugin>
+        </visual>
+    </gazebo>
+    <gazebo reference="HL_foot">
+        <visual>
+            <plugin name="drawForcePlugin" filename="libunitreeDrawForcePlugin.so">
+                <topicName>HL_foot_contact</topicName>
+            </plugin>
+        </visual>
+    </gazebo> -->
+    </xacro:if>
     <xacro:if value="${int(ros_version) == 2}">
     <gazebo reference="imu_link">
@@ -163,5 +285,5 @@
         <kd  value="1.0"/>
     </gazebo>
-    <!-- RL leg -->
+    <!-- HL leg -->
     <gazebo reference="HL_HIP">
         <mu1>0.2</mu1>
@@ -187,5 +309,5 @@
         <kd  value="1.0"/>
     </gazebo>
-    <!-- RR leg -->
+    <!-- HR leg -->
     <gazebo reference="HR_HIP">
         <mu1>0.2</mu1>

File: src/robots/lite3_description/xacro/robot.xacro (robot description, xacro)
@@ -1,8 +1,5 @@
 <?xml version="1.0"?>
 <robot name="lite3" xmlns:xacro="http://www.ros.org/wiki/xacro">
-    <!-- <xacro:include filename="$(find lite3_description)/xacro/gazebo.xacro"/>
-    <xacro:include filename="$(find lite3_description)/xacro/body.xacro"/>
-    <xacro:include filename="$(find lite3_description)/xacro/transmission.xacro"/> -->
-    <xacro:include filename="$(find lite3_description)/urdf/Lite3.urdf"/>
+    <xacro:include filename="$(find lite3_description)/urdf/lite3.urdf"/>
     <xacro:include filename="$(find lite3_description)/xacro/gazebo.xacro"/>
 </robot>

Commit message: Fix:Update Lite3 URDF to align with official version

File: src/robots/lite3_description/urdf/lite3.urdf (robot description, URDF)
Before this commit: robot Lite3, 19 links, 18 joints
Links:
- removed link base
- link FL_HIP: geometry collision cylinder length=0.15 radius=0.04; visual mesh filename=package://lite3_description/meshes/fl_hip.STL
- link FL_SHANK: geometry collision cylinder length=0.10 radius=0.015; collision cylinder length=0.12 radius=0.015
- link FL_THIGH: geometry collision box size=0.04 0.045 0.2; visual mesh filename=package://lite3_description/meshes/fl_thigh.STL
- link FR_HIP: geometry collision cylinder length=0.15 radius=0.04; visual mesh filename=package://lite3_description/meshes/fr_hip.STL
- link FR_SHANK: geometry collision cylinder length=0.10 radius=0.015; collision cylinder length=0.12 radius=0.015
- link FR_THIGH: geometry collision box size=0.04 0.045 0.2; visual mesh filename=package://lite3_description/meshes/fr_thigh.STL
- link HL_HIP: geometry collision cylinder length=0.15 radius=0.04; visual mesh filename=package://lite3_description/meshes/hl_hip.STL
- link HL_SHANK: geometry collision cylinder length=0.10 radius=0.015; collision cylinder length=0.12 radius=0.015
- link HL_THIGH: geometry collision box size=0.04 0.045 0.2; visual mesh filename=package://lite3_description/meshes/hl_thigh.STL
- link HR_HIP: geometry collision cylinder length=0.15 radius=0.04; visual mesh filename=package://lite3_description/meshes/hr_hip.STL
- link HR_SHANK: geometry collision cylinder length=0.10 radius=0.015; collision cylinder length=0.12 radius=0.015
- link HR_THIGH: geometry collision box size=0.04 0.045 0.2; visual mesh filename=package://lite3_description/meshes/hr_thigh.STL
- link TORSO: geometry collision box size=0.25 0.2 0.12; collision box size=0.5 0.1 0.12
Joints:
- removed joint FL_HipX
- removed joint FL_HipY
- removed joint FL_Knee
- removed joint FR_HipX
- removed joint FR_HipY
- removed joint FR_Knee
- removed joint HL_HipX
- removed joint HL_HipY
- removed joint HL_Knee
- removed joint HR_HipX
- removed joint HR_HipY
- removed joint HR_Knee
- removed joint floating_base
- added joint FL_HipX_joint: type revolute, parent TORSO, child FL_HIP, origin xyz=0.1745 0.062 0 rpy=0 0 0, axis -1 0 0, limit lower=-0.523 upper=0.523 effort=24 velocity=26.2
- added joint FL_HipY_joint: type revolute, parent FL_HIP, child FL_THIGH, origin xyz=0 0.09735 0 rpy=0 0 0, axis 0 -1 0, limit lower=-2.67 upper=0.314 effort=24 velocity=26.2
- added joint FL_Knee_joint: type revolute, parent FL_THIGH, child FL_SHANK, origin xyz=0 0 -0.20 rpy=0 0 0, axis 0 -1 0, limit lower=0.524 upper=2.792 effort=36 velocity=17.3
- added joint FR_HipX_joint: type revolute, parent TORSO, child FR_HIP, origin xyz=0.1745 -0.062 0 rpy=0 0 0, axis -1 0 0, limit lower=-0.523 upper=0.523 effort=24 velocity=26.2
- added joint FR_HipY_joint: type revolute, parent FR_HIP, child FR_THIGH, origin xyz=0 -0.09735 0 rpy=0 0 0, axis 0 -1 0, limit lower=-2.67 upper=0.314 effort=24 velocity=26.2
- added joint FR_Knee_joint: type revolute, parent FR_THIGH, child FR_SHANK, origin xyz=0 0 -0.20 rpy=0 0 0, axis 0 -1 0, limit lower=0.524 upper=2.792 effort=36 velocity=17.3
- added joint HL_HipX_joint: type revolute, parent TORSO, child HL_HIP, origin xyz=-0.1745 0.062 0 rpy=0 0 0, axis -1 0 0, limit lower=-0.523 upper=0.523 effort=24 velocity=26.2
- added joint HL_HipY_joint: type revolute, parent HL_HIP, child HL_THIGH, origin xyz=0 0.09735 0 rpy=0 0 0, axis 0 -1 0, limit lower=-2.67 upper=0.314 effort=24 velocity=26.2
- added joint HL_Knee_joint: type revolute, parent HL_THIGH, child HL_SHANK, origin xyz=0 0 -0.20 rpy=0 0 0, axis 0 -1 0, limit lower=0.524 upper=2.792 effort=36 velocity=17.3
- added joint HR_HipX_joint: type revolute, parent TORSO, child HR_HIP, origin xyz=-0.1745 -0.062 0 rpy=0 0 0, axis -1 0 0, limit lower=-0.523 upper=0.523 effort=24 velocity=26.2
- added joint HR_HipY_joint: type revolute, parent HR_HIP, child HR_THIGH, origin xyz=0 -0.09735 0 rpy=0 0 0, axis 0 -1 0, limit lower=-2.67 upper=0.314 effort=24 velocity=26.2
- added joint HR_Knee_joint: type revolute, parent HR_THIGH, child HR_SHANK, origin xyz=0 0 -0.20 rpy=0 0 0, axis 0 -1 0, limit lower=0.524 upper=2.792 effort=36 velocity=17.3

File: src/robots/lite3_description/xacro/gazebo.xacro (robot description, xacro)
@@ -212,7 +212,7 @@
         </xacro:macro>
         <xacro:macro name="leg_joints" params="prefix">
-            <xacro:joint_interface joint_name="${prefix}_HipX" torque_limit="${HipX_torque_max}"/>
-            <xacro:joint_interface joint_name="${prefix}_HipY" torque_limit="${HipY_torque_max}"/>
-            <xacro:joint_interface joint_name="${prefix}_Knee" torque_limit="${Knee_torque_max}"/>
+            <xacro:joint_interface joint_name="${prefix}_HipX_joint" torque_limit="${HipX_torque_max}"/>
+            <xacro:joint_interface joint_name="${prefix}_HipY_joint" torque_limit="${HipY_torque_max}"/>
+            <xacro:joint_interface joint_name="${prefix}_Knee_joint" torque_limit="${Knee_torque_max}"/>
         </xacro:macro>
         <xacro:leg_joints prefix="FR"/>
