Commit message: fix lite3

File: src/robots/lite3_description/xacro/gazebo.xacro (robot description, xacro)
@@ -1,7 +1,7 @@
 <?xml version="1.0"?>
 <robot xmlns:xacro="http://www.ros.org/wiki/xacro">
-    <xacro:property name="HipX_torque_max" value="40"/>
-    <xacro:property name="HipY_torque_max" value="40"/>
-    <xacro:property name="Knee_torque_max" value="65"/>
+    <xacro:property name="HipX_torque_max" value="30"/>
+    <xacro:property name="HipY_torque_max" value="30"/>
+    <xacro:property name="Knee_torque_max" value="30"/>
     <xacro:property name="ros_version" value="$(env ROS_VERSION)" />
     <xacro:if value="${int(ros_version) == 2}">
